File: DIMECRES_C_retrovisors.kicad_sch (KiCad schematic)
At the start: 62 parts, among them J1 Conn_Entrada, J2 DE9_Pins, J3 Conn_01x05_Pin, J4 Botonera, J5 SENSOR, J6 Intermitent, J7 Calentador, Q1 DTC144E, Q2 DTC144E, Q3 DTC144E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

Commit message: CorrecionV3
Parts:
- removed J1: Conn_Entrada, symbol Connector:Conn_01x02_Pin
- removed J4: Botonera, symbol Connector:Conn_01x06_Pin
- removed J5: SENSOR, symbol Connector:Conn_01x04_Pin
- removed J6: Intermitent, symbol Connector:Conn_01x02_Pin
- removed J7: Calentador, symbol Connector:Conn_01x02_Pin
- added J10: Vbat, symbol Connector:Screw_Terminal_01x02
- added J4: Motor3, symbol Connector:Screw_Terminal_01x02
- added J6: Intermitente, symbol Connector:Screw_Terminal_01x02
- added J7: Calentador, symbol Connector:Screw_Terminal_01x02
- added J8: Motor2, symbol Connector:Screw_Terminal_01x02
- added J9: Motor1, symbol Connector:Screw_Terminal_01x02
- added U1: ~, symbol PracticasKiCad:Botonera_Retrovisor
- added U10: ~, symbol PracticasKiCad:Sensor_SR55
Connections:
- net Down: now also U1.4
- net GND: now also J10.2 (Pin_2), J6.2 (Pin_2), J7.2 (Pin_2), U10.3 (A_OUT)
- net Heat: now also U1.2
- net Left: now also U1.5
- net Right: now also U1.6
- net SCL: now also U10.2 (T)
- net SDA: now also U10.4 (-U)
- net Un/Fold: now also U1.1
- net Up: now also U1.3
- net Vbat: now also J10.1 (Pin_1), U10.1 (+U)
- net at U9.3: now also J6.1 (Pin_1)
- net at U8.3: now also J7.1 (Pin_1)
- net CANH: no longer names the net of J2.7, R7.1, U5.7 (CANH)
- net CANL: no longer names the net of J2.2, R6.2, U5.6 (CANL)
- net Intermitent renamed Intermitente
- net Motor1A: no longer names the net of U4.2 (OUT1)
- net Motor1A: now also J9.1 (Pin_1)
- net Motor1B: no longer names the net of U4.3 (OUT2)
- net Motor1B: now also J9.2 (Pin_2)
- net Motor2A: no longer names the net of SW1.10
- net Motor2A: now also J8.1 (Pin_1)
- net Motor2B: no longer names the net of SW1.3
- net Motor2B: now also J8.2 (Pin_2)
- net Motor3A: no longer names the net of SW1.8
- net Motor3A: now also J4.1 (Pin_1)
- net Motor3B: no longer names the net of SW1.5
- net Motor3B: now also J4.2 (Pin_2)
Other:
- note added: "CIRCUIT OSCIL·LADOR"
- note removed: "ALIMENTACIO OPAMP"
- note removed: "BUS CAN"
- note removed: "OSCILLATOR CIRCUIT"
- moved on the sheet: C11, C12, C13, C15, C16, C17, C7, C8, D2, J2, Q1, Q2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

Commit message: Update DIMECRES_C_retrovisors.kicad_sch
Parts:
- C4: value 10n -> 100n
- C5: value 100n -> 100u
Connections:
- net Vcc: no longer C4.1
- net at C2.1, L1.2, R2.2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: now also C4.1
Other:
- moved on the sheet: C3, C4, C5, R4, R5, U2

Commit message: Update DIMECRES_C_retrovisors.kicad_sch
Parts:
- removed R3: 5, symbol Device:R
- added C18: 1n, symbol Device:C
- C1: value 100u -> 120u
- C2: value 220u -> 470u
- C5: value 100u -> 22u
- L1: value 47u -> 33u
Connections:
- net GND: now also U10.4 (A_OUT); no longer U10.3 (A_OUT), U9.1
- net SDA: now also U10.3 (-U); no longer U10.4 (-U)
- net at R1.2, R2.1, U3.4 (FB): now also C18.1
- net at C2.1, C4.1, L1.2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: now also C18.2
- no-connect marks 4 -> 6

Commit message: Update DIMECRES_C_retrovisors.kicad_sch
Parts:
- removed U1: ~, symbol PracticasKiCad:Botonera_Retrovisor
- added SW2, SW3, SW4, SW5, SW6, SW7: SW_Push, symbol Switch:SW_Push
Connections:
- net Down: now also SW5.2
- net Heat: now also SW3.2
- net Left: now also SW6.2
- net Right: now also SW7.2
- net Un/Fold: now also SW2.2
- net Up: now also SW4.2
- net Vcc: now also SW2.1, SW3.1, SW4.1, SW5.1, SW6.1, SW7.1

Commit message: .2
Connections:
- net ENA is gone; now on net EN1: U7.17 (CCP1/RC2)
- net ENB is gone; now on net EN2/3: U7.21 (C2IN+/PSP2/RD2)
- net GND: now also U5.8 (STB)
- net STB: no longer U5.8 (STB)
- net Motor2+: now reaches J8.1 (Pin_1), SW1.10
- net Motor2-: now reaches J8.2 (Pin_2), SW1.3
- net Motor2-: now also J4.2 (Pin_2), SW1.5
- net Motor23-: now reaches SW1.4, U4.14 (OUT4)
- net Motor3+: now reaches J4.1 (Pin_1), SW1.8
- net Motor23+: now reaches SW1.9, U4.13 (OUT3)
- net Motor1+: now reaches J9.1 (Pin_1), U4.2 (OUT1)
- net Motor1-: now reaches J9.2 (Pin_2), U4.3 (OUT2)
- net Down renamed B_Down
- net Heat renamed B_Heat
- net Left renamed B_Left
- net Right renamed B_Right
- net Un/Fold renamed B_Un/Fold
- net Up renamed B_Up
Other:
- moved on the sheet: C11, J4, J8, J9, SW1

Commit message: Up. sch.
Parts:
- removed R4: 364, symbol Device:R
- removed R5: 121, symbol Device:R
- removed U10: ~, symbol PracticasKiCad:Sensor_SR55
- removed U2: LM1117DT-ADJ, Package_TO_SOT_SMD:TO-252-3_TabPin2, symbol Regulator_Linear:LM1117DT-ADJ
- added C19: 4u7, symbol Device:C
- added C20: 100n, symbol Device:C
- added R3: 10k, symbol Device:R
- added U1: ~, symbol PracticasKiCad:Sensor_CH201
- added U10: LM1117DT-5.0, Package_TO_SOT_SMD:TO-252-3_TabPin2, symbol Regulator_Linear:LM1117DT-5.0
- added U2: ~, symbol PracticasKiCad:ADM7160
- C3: value 10n -> 4u7
- R10, R11: value 4k7 -> 2k2
Connections:
- net GND: now also C19.2, C20.2, U1.5 (VSS), U10.1 (GND), U2.2 (GND)
- net Vcc: now also C3.1, U10.2 (VO), U2.1 (Vin), U2.3 (EN); no longer R10.1, R11.1
- net at C18.2, C2.1, C4.1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: now also U10.3 (VI)
- net at U7.29 (P1C/PSP6/RD6): now also U1.3 (PROG)
- net at U7.30 (P1D/PSP7/RD7): now also U1.1 (INT)
- net SCL: no longer names the net of R10.2, U7.18 (SCL/SCK/RC3)
- net SCL: now also U1.2 (SCL)
- net SDA: no longer names the net of R11.2, U7.23 (SDA/SDI/RC4)
- net SDA: now also U1.4 (SDA)
- net XTAL1: no longer names the net of C12.1, U7.13 (OSC1/CLKI/RA7), Y1.1
- net XTAL2: no longer names the net of C13.1, U7.14 (OSC2/CLKO/RA6), Y1.2
- new net Rst_N: R3.2, U1.8 (RST_N)
- new net Vdd: C19.1, C20.1, R10.1, R11.1, R3.1, U1.6 (VDD), U1.7 (AVDD), U2.5 (Vout)
Other:
- note added: "Colocar capacitat el més aprop de Vdd Avdd"
- moved on the sheet: C12, C13, C14, C9, R10, R11, U7, Y1

Commit message: Update DIMECRES_C_retrovisors.kicad_sch
Parts:
- removed R8, R9: 50m, symbol Device:R_Shunt
- added D3, D5, D6: 1N5817, Diode_THT:D_DO-41_SOD81_P10.16mm_Horizontal, symbol Diode:1N5817
- added R4, R5: 50m, symbol Device:R
Connections:
- net GNDPWR: now also R12.1, R17.1, R4.2, R5.2
- net SENSE_A: now also R14.1, R4.1
- net SENSE_B: now also R16.1, R5.1
- net Vbat: now also D3.1 (K), D5.1 (K), D6.1 (K)
- net at Q2.3 (C), U9.2: now also D5.2 (A)
- net at Q1.3 (C), SW1.1: now also D6.2 (A)
- net at Q3.3 (C), U8.2: now also D3.2 (A)
Other:
- moved on the sheet: C15, C16

Commit message: Up de tot
Parts:
- added J5: DE9_Pins, Connector_Dsub:DSUB-9_Socket_Horizontal_P2.77x2.54mm_EdgePinOffset9.40mm, symbol Connector:DE9_Pins
- added R8: 0, symbol Device:R
- C5: value 22u -> 100u
- J10, J4, J6, J7, J8, J9: footprint (none) -> Connector_TE-Connectivity:TE_826576-2_1x02_P3.96mm_Vertical
- J2: footprint (none) -> Connector_Dsub:DSUB-9_Socket_Horizontal_P2.77x2.54mm_EdgePinOffset9.40mm
- J3: footprint (none) -> Connector_PinHeader_2.54mm:PinHeader_1x05_P2.54mm_Vertical
- U4: footprint Package_TO_SOT_THT:TO-220-15_P2.54x2.54mm_StaggerOdd_Lead4.58mm_Vertical -> Package_TO_SOT_THT:TO-220-15_P2.54x5.08mm_StaggerOdd_Lead4.58mm_Vertical
Connections:
- net AngleMort: now also U7.8 (AN5/~{RD}/RE0); no longer U7.26 (DT/RX/RC7)
- net GND: now also J5.5, R8.1
- net GNDPWR: now also R8.2
- net Intermitente: now also U7.9 (C1OUT/AN6/~{WR}/RE1); no longer U7.25 (CK/TX/RC6)
- net S_SDA: now reaches R11.2, U1.4 (SDA), U7.23 (SDA/SDI/RC4)
- net CAN-: now reaches J2.2, R6.2, U5.6 (CANL)
- net CAN+: now reaches J2.7, R7.1, U5.7 (CANH)
- net S_SCL: now reaches R10.2, U1.2 (SCL), U7.18 (SCL/SCK/RC3)
- net S_PROG: now reaches U1.3 (PROG), U7.29 (P1C/PSP6/RD6)
- net S_INT: now reaches U1.1 (INT), U7.30 (P1D/PSP7/RD7)
- new net Tx: J5.3
- no-connect marks 6 -> 8
Other:
- note added: "REGULADOR 1.8V"
- note added: "Unificacio gnd-gndpwr, no montar r"
- moved on the sheet: C10, C12, C13, C14, C19, C20, C3, C6, C9, J2, R10, R11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
