File: DIMECRES_C_retrovisors.kicad_sch (KiCad schematic)
At the start: 84 parts, among them J10 Vbat, J2 DE9_Pins, J3 Conn_01x05_Pin, J4 Motor3, J5 DE9_Pins, J6 Intermitente, J7 Calentador, J8 Motor2, J9 Motor1, Q1 DTC144E, Q2 DTC144E, Q3 DTC144E, SW1 SW_DPDT_G6S, SW10 SW_Push, SW2 SW_Push, SW3 SW_Push, SW4 SW_Push, SW5 SW_Push, SW6 SW_Push, SW7 SW_Push, SW8 FN01B, SW9 FN01B, U1 CH201, U10 LM1117DT-5.0, U2 ADM7160, U3 LM2596S-ADJ, U4 L298N, U5 MCP2551-I-SN, U6 ADA4511-2, U7 PIC18F4480-IP, Y1 Crystal

Commit message: lop
Parts:
- R22, R23, R24: footprint (none) -> Resistor_SMD:R_0805_2012Metric_Pad1.20x1.40mm_HandSolder
Changed lines of the file:
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@@
 			)
 		)
-		(property "Footprint" ""
+		(property "Footprint" "Resistor_SMD:R_0805_2012Metric_Pad1.20x1.40mm_HandSolder"
 			(at 214.122 269.24 90)
 			(effects
@@
 			)
 		)
-		(property "Footprint" ""
+		(property "Footprint" "Resistor_SMD:R_0805_2012Metric_Pad1.20x1.40mm_HandSolder"
 			(at 335.407 245.745 90)
 			(effects
@@
 			)
 		)
-		(property "Footprint" ""
+		(property "Footprint" "Resistor_SMD:R_0805_2012Metric_Pad1.20x1.40mm_HandSolder"
 			(at 356.362 102.87 90)
 			(effects

Commit message: Proimeres correccions
Parts:
- removed C7: 100n, Capacitor_SMD:C_1206_3216Metric_Pad1.33x1.80mm_HandSolder, symbol Device:C
- added C6: 470U, Capacitor_THT:CP_Radial_D6.3mm_P2.50mm, symbol Device:C
- added D10, D11, D12, D13, D14, D7, D8, D9: 1N5822, Diode_THT:D_DO-201AD_P15.24mm_Horizontal, symbol Diode:1N5822
Connections:
- net Act_Rele_M2/M3: now also U7.17 (CCP1/RC2); no longer U7.10 (C2OUT/AN7/~{CS}/RE2)
- net B_Up: now also U7.24 (SDO/RC5); no longer U7.22 (C2IN-/PSP3/RD3)
- net Calentador: now also U7.38 (RB5/KBI1/PGM); no longer U7.5 (RA3/AN3/Vref+)
- net EN1: now also U7.6 (RA4/TOCKI); no longer U7.17 (CCP1/RC2)
- net EN2/3: now also U7.9 (C1OUT/AN6/~{WR}/RE1); no longer U7.21 (C2IN+/PSP2/RD2)
- net GNDPWR: now also C6.2, D11.2 (A), D12.2 (A), D13.2 (A), D14.2 (A)
- net IN1A: now also U7.5 (RA3/AN3/Vref+); no longer U7.15 (T13CKI/T1OSO/RC0)
- net IN1B: now also U7.7 (RA5/ANA4/~{SS}/HLVDIN); no longer U7.16 (T1OSI/RC1)
- net IN2/3A: now also U7.8 (AN5/~{RD}/RE0); no longer U7.19 (C1IN+/PSP0/RD0)
- net IN2/3B: now also U7.10 (C2OUT/AN7/~{CS}/RE2); no longer U7.20 (C1IN-/PSP1/RD1)
- net Intermitente: now also U7.37 (RB4/KBI0/AN9); no longer U7.9 (C1OUT/AN6/~{WR}/RE1)
- net Motor1A: now also D11.1 (K), D7.2 (A)
- net Motor1B: now also D12.1 (K), D8.2 (A)
- net Motor23A: now also D13.1 (K), D9.2 (A)
- net Motor23B: now also D10.2 (A), D14.1 (K)
- net S_INT: now also U7.22 (C2IN-/PSP3/RD3); no longer U7.34 (RB1/INT1/AN8)
- net S_PROG: now also U7.21 (C2IN+/PSP2/RD2); no longer U7.24 (SDO/RC5)
- net Vbat: now also C6.1, D10.1 (K), D7.1 (K), D8.1 (K), D9.1 (K)
Other:
- note added: "Les capacitats c8, c17 s'han de colocar aprop dels dispositius"
- note removed: "Les capacitats c7, c8, c17 s'han de colocar aprop dels dispositius"
- moved on the sheet: C11, C17, C8, D6, J4, J9, Q1, R24, U4, U6C

Commit message: planos vcc
Connections:
- net Act_Rele_M2/M3: now also U7.19 (C1IN+/PSP0/RD0); no longer U7.17 (CCP1/RC2)
- net Intermitente: now also U7.20 (C1IN-/PSP1/RD1); no longer U7.37 (RB4/KBI0/AN9)
Changed lines of the file:
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@@
 	)
 	(no_connect
-		(at 145.415 160.655)
+		(at 141.605 142.875)
 	)
 	(no_connect
@@
 	)
 	(no_connect
-		(at 145.415 163.195)
+		(at 76.835 178.435)
 	)
 	(no_connect
@@
 	(global_label "Act_Rele_M2{slash}M3"
 		(shape input)
-		(at 141.605 142.875 0)
+		(at 145.415 160.655 0)
 		(fields_autoplaced yes)
 		(effects
@@
 		)
 		(property "Intersheetrefs" "${INTERSHEET_REFS}"
-			(at 160.193 142.875 0)
+			(at 164.003 160.655 0)
 			(effects
 				(font
@@
 	(global_label "Intermitente"
 		(shape input)
-		(at 76.835 178.435 180)
+		(at 145.415 163.195 0)
 		(fields_autoplaced yes)
 		(effects
@@
 				(size 1.27 1.27)
 			)
-			(justify right)
+			(justify left)
 		)
 		(property "Intersheetrefs" "${INTERSHEET_REFS}"
-			(at 62.4198 178.435 0)
+			(at 159.8302 163.195 0)
 			(effects
 				(font
 					(size 1.27 1.27)
 				)
-				(justify right)
+				(justify left)
 				(hide yes)
 			)

Commit message: correccion errores
Connections:
- net AngleMort: now also U7.38 (RB5/KBI1/PGM); no longer U7.4 (RA2/AN2/Vref-)
- net Calentador: now also U7.4 (RA2/AN2/Vref-); no longer U7.38 (RB5/KBI1/PGM)
Changed lines of the file:
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@@
 	(global_label "AngleMort"
 		(shape input)
+		(at 79.375 180.975 180)
+		(fields_autoplaced yes)
+		(effects
+			(font
+				(size 1.27 1.27)
+			)
+			(justify right)
+		)
+		(property "Intersheetrefs" "${INTERSHEET_REFS}"
+			(at 67.1371 180.975 0)
+			(effects
+				(font
+					(size 1.27 1.27)
+				)
+				(justify right)
+				(hide yes)
+			)
+		)
+	)
+	(global_label "SENSE_B"
+		(shape input)
+		(at 350.52 170.18 180)
+		(fields_autoplaced yes)
+		(effects
+			(font
+				(size 1.27 1.27)
+			)
+			(justify right)
+		)
+		(property "Intersheetrefs" "${INTERSHEET_REFS}"
+			(at 339.2497 170.18 0)
+			(effects
+				(font
+					(size 1.27 1.27)
+				)
+				(justify right)
+				(hide yes)
+			)
+		)
+	)
+	(global_label "Vbat"
+		(shape input)
+		(at 301.625 212.725 180)
+		(fields_autoplaced yes)
+		(effects
+			(font
+				(size 1.27 1.27)
+			)
+			(justify right)
+		)
+		(property "Intersheetrefs" "${INTERSHEET_REFS}"
+			(at 294.5275 212.725 0)
+			(effects
+				(font
+					(size 1.27 1.27)
+				)
+				(justify right)
+				(hide yes)
+			)
+		)
+	)
+	(global_label "B_Up"
+		(shape input)
+		(at 145.415 150.495 0)
+		(fields_autoplaced yes)
+		(effects
+			(font
+				(size 1.27 1.27)
+			)
+			(justify left)
+		)
+		(property "Intersheetrefs" "${INTERSHEET_REFS}"
+			(at 153.1173 150.495 0)
+			(effects
+				(font
+					(size 1.27 1.27)
+				)
+				(justify left)
+				(hide yes)
+			)
+		)
+	)
+	(global_label "SENSE_A"
+		(shape input)
+		(at 286.385 78.74 270)
+		(fields_autoplaced yes)
+		(effects
+			(font
+				(size 1.27 1.27)
+			)
+			(justify right)
+		)
+		(property "Intersheetrefs" "${INTERSHEET_REFS}"
+			(at 286.385 89.8289 90)
+			(effects
+				(font
+					(size 1.27 1.27)
+				)
+				(justify right)
+				(hide yes)
+			)
+		)
+	)
+	(global_label "Vcc"
+		(shape input)
+		(at 246.38 35.56 90)
+		(fields_autoplaced yes)
+		(effects
+			(font
+				(size 1.27 1.27)
+			)
+			(justify left)
+		)
+		(property "Intersheetrefs" "${INTERSHEET_REFS}"
+			(at 246.38 29.309 90)
+			(effects
+				(font
+					(size 1.27 1.27)
+				)
+				(justify left)
+				(hide yes)
+			)
+		)
+	)
+	(global_label "Act_Rele_M2{slash}M3"
+		(shape input)
+		(at 145.415 160.655 0)
+		(fields_autoplaced yes)
+		(effects
+			(font
+				(size 1.27 1.27)
+			)
+			(justify left)
+		)
+		(property "Intersheetrefs" "${INTERSHEET_REFS}"
+			(at 164.003 160.655 0)
+			(effects
+				(font
+					(size 1.27 1.27)
+				)
+				(justify left)
+				(hide yes)
+			)
+		)
+	)
+	(global_label "B_Un{slash}Fold"
+		(shape input)
+		(at 50.8 71.12 0)
+		(fields_autoplaced yes)
+		(effects
+			(font
+				(size 1.27 1.27)
+			)
+			(justify left)
+		)
+		(property "Intersheetrefs" "${INTERSHEET_REFS}"
+			(at 63.8846 71.12 0)
+			(effects
+				(font
+					(size 1.27 1.27)
+				)
+				(justify left)
+				(hide yes)
+			)
+		)
+	)
+	(global_label "PGD"
+		(shape input)
+		(at 79.375 186.055 180)
+		(fields_autoplaced yes)
+		(effects
+			(font
+				(size 1.27 1.27)
+			)
+			(justify right)
+		)
+		(property "Intersheetrefs" "${INTERSHEET_REFS}"
+			(at 72.5798 186.055 0)
+			(effects
+				(font
+					(size 1.27 1.27)
+				)
+				(justify right)
+				(hide yes)
+			)
+		)
+	)
+	(global_label "Vcc"
+		(shape input)
+		(at 345.44 63.5 180)
+		(fields_autoplaced yes)
+		(effects
+			(font
+				(size 1.27 1.27)
+			)
+			(justify right)
+		)
+		(property "Intersheetrefs" "${INTERSHEET_REFS}"
+			(at 339.189 63.5 0)
+			(effects
+				(font
+					(size 1.27 1.27)
+				)
+				(justify right)
+				(hide yes)
+			)
+		)
+	)
+	(global_label "Calentador"
+		(shape input)
 		(at 79.375 147.955 180)
 		(fields_autoplaced yes)
@@
 		)
 		(property "Intersheetrefs" "${INTERSHEET_REFS}"
-			(at 67.1371 147.955 0)
-			(effects
-				(font
-					(size 1.27 1.27)
-				)
-				(justify right)
-				(hide yes)
-			)
-		)
-	)
-	(global_label "SENSE_B"
-		(shape input)
-		(at 350.52 170.18 180)
-		(fields_autoplaced yes)
-		(effects
-			(font
-				(size 1.27 1.27)
-			)
-			(justify right)
-		)
-		(property "Intersheetrefs" "${INTERSHEET_REFS}"
-			(at 339.2497 170.18 0)
-			(effects
-				(font
-					(size 1.27 1.27)
-				)
-				(justify right)
-				(hide yes)
-			)
-		)
-	)
-	(global_label "Vbat"
-		(shape input)
-		(at 301.625 212.725 180)
-		(fields_autoplaced yes)
-		(effects
-			(font
-				(size 1.27 1.27)
-			)
-			(justify right)
-		)
-		(property "Intersheetrefs" "${INTERSHEET_REFS}"
-			(at 294.5275 212.725 0)
-			(effects
-				(font
-					(size 1.27 1.27)
-				)
-				(justify right)
-				(hide yes)
-			)
-		)
-	)
-	(global_label "B_Up"
-		(shape input)
-		(at 145.415 150.495 0)
-		(fields_autoplaced yes)
-		(effects
-			(font
-				(size 1.27 1.27)
-			)
-			(justify left)
-		)
-		(property "Intersheetrefs" "${INTERSHEET_REFS}"
-			(at 153.1173 150.495 0)
-			(effects
-				(font
-					(size 1.27 1.27)
-				)
-				(justify left)
-				(hide yes)
-			)
-		)
-	)
-	(global_label "SENSE_A"
-		(shape input)
-		(at 286.385 78.74 270)
-		(fields_autoplaced yes)
-		(effects
-			(font
-				(size 1.27 1.27)
-			)
-			(justify right)
-		)
-		(property "Intersheetrefs" "${INTERSHEET_REFS}"
-			(at 286.385 89.8289 90)
-			(effects
-				(font
-					(size 1.27 1.27)
-				)
-				(justify right)
-				(hide yes)
-			)
-		)
-	)
-	(global_label "Vcc"
-		(shape input)
-		(at 246.38 35.56 90)
-		(fields_autoplaced yes)
-		(effects
-			(font
-				(size 1.27 1.27)
-			)
-			(justify left)
-		)
-		(property "Intersheetrefs" "${INTERSHEET_REFS}"
-			(at 246.38 29.309 90)
-			(effects
-				(font
-					(size 1.27 1.27)
-				)
-				(justify left)
-				(hide yes)
-			)
-		)
-	)
-	(global_label "Act_Rele_M2{slash}M3"
-		(shape input)
-		(at 145.415 160.655 0)
-		(fields_autoplaced yes)
-		(effects
-			(font
-				(size 1.27 1.27)
-			)
-			(justify left)
-		)
-		(property "Intersheetrefs" "${INTERSHEET_REFS}"
-			(at 164.003 160.655 0)
-			(effects
-				(font
-					(size 1.27 1.27)
-				)
-				(justify left)
-				(hide yes)
-			)
-		)
-	)
-	(global_label "B_Un{slash}Fold"
-		(shape input)
-		(at 50.8 71.12 0)
-		(fields_autoplaced yes)
-		(effects
-			(font
-				(size 1.27 1.27)
-			)
-			(justify left)
-		)
-		(property "Intersheetrefs" "${INTERSHEET_REFS}"
-			(at 63.8846 71.12 0)
-			(effects
-				(font
-					(size 1.27 1.27)
-				)
-				(justify left)
-				(hide yes)
-			)
-		)
-	)
-	(global_label "PGD"
-		(shape input)
-		(at 79.375 186.055 180)
-		(fields_autoplaced yes)
-		(effects
-			(font
-				(size 1.27 1.27)
-			)
-			(justify right)
-		)
-		(property "Intersheetrefs" "${INTERSHEET_REFS}"
-			(at 72.5798 186.055 0)
-			(effects
-				(font
-					(size 1.27 1.27)
-				)
-				(justify right)
-				(hide yes)
-			)
-		)
-	)
-	(global_label "Vcc"
-		(shape input)
-		(at 345.44 63.5 180)
-		(fields_autoplaced yes)
-		(effects
-			(font
-				(size 1.27 1.27)
-			)
-			(justify right)
-		)
-		(property "Intersheetrefs" "${INTERSHEET_REFS}"
-			(at 339.189 63.5 0)
-			(effects
-				(font
-					(size 1.27 1.27)
-				)
-				(justify right)
-				(hide yes)
-			)
-		)
-	)
-	(global_label "Calentador"
-		(shape input)
-		(at 79.375 180.975 180)
-		(fields_autoplaced yes)
-		(effects
-			(font
-				(size 1.27 1.27)
-			)
-			(justify right)
-		)
-		(property "Intersheetrefs" "${INTERSHEET_REFS}"
-			(at 66.1091 180.975 0)
-			(effects
-				(font
+			(at 66.1091 147.955 0)
+			(effects
+				(font

Commit message: kk
Parts:
- added C23: 100n, Capacitor_SMD:C_1206_3216Metric_Pad1.33x1.80mm_HandSolder, symbol Device:C
- added R25, R26: 1K, Resistor_SMD:R_1206_3216Metric_Pad1.30x1.75mm_HandSolder, symbol Device:R
- added U8: LSF0002, symbol PracticasKiCad:LSF0002
- R10, R11: value 2k2 -> 1K
Connections:
- net GND: now also C23.2, U8.1 (GND)
- net S_SCL: now also R26.2, U8.2 (A1); no longer R10.2, U1.2 (SCL)
- net S_SDA: now also R25.2, U8.3 (A2); no longer R11.2, U1.4 (SDA)
- net Vcc: now also R25.1, R26.1
- net Vdd: now also C23.1, U8.6 (VBIAS)
- new net: R11.2, U1.4 (SDA), U8.4 (B2)
- new net: R10.2, U1.2 (SCL), U8.5 (B1)
Other:
- moved on the sheet: C16, C20, C22, D3, J5, J7, Q3, R10, R11, R22, R3, R8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

Commit message: De to
Parts:
- C23: footprint Capacitor_SMD:C_1206_3216Metric_Pad1.33x1.80mm_HandSolder -> Capacitor_SMD:C_0805_2012Metric_Pad1.18x1.45mm_HandSolder
- R10, R11, R25, R26: footprint Resistor_SMD:R_1206_3216Metric_Pad1.30x1.75mm_HandSolder -> Resistor_SMD:R_0805_2012Metric_Pad1.20x1.40mm_HandSolder
- SW2: value SW_Push -> UN/FOLD
- SW3: value SW_Push -> HEAT
- SW4: value SW_Push -> UP
- SW5: value SW_Push -> DOWN
- SW6: value SW_Push -> LEFT
- SW7: value SW_Push -> RIGHT
- U10: footprint Package_TO_SOT_SMD:TO-252-3_TabPin2 -> Package_TO_SOT_SMD:TO-263-3_TabPin2
- U8: footprint (none) -> PracticasKiCad:LSF0002
Other:
- moved on the sheet: SW2
Changed lines of the file:
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@@
 	(wire
 		(pts
-			(xy 33.02 67.945) (xy 38.1 67.945)
+			(xy 33.02 65.405) (xy 38.1 65.405)
 		)
 		(stroke
@@
 	(wire
 		(pts
-			(xy 53.34 67.945) (xy 48.26 67.945)
+			(xy 48.26 65.405) (xy 53.975 65.405)
 		)
 		(stroke
@@
 	(wire
 		(pts
-			(xy 33.02 67.945) (xy 33.02 75.565)
+			(xy 33.02 65.405) (xy 33.02 75.565)
 		)
 		(stroke
@@
 	(global_label "B_Un{slash}Fold"
 		(shape input)
-		(at 53.34 67.945 0)
+		(at 53.975 65.405 0)
 		(fields_autoplaced yes)
 		(effects
@@
 		)
 		(property "Intersheetrefs" "${INTERSHEET_REFS}"
-			(at 66.4246 67.945 0)
+			(at 67.0596 65.405 0)
 			(effects
 				(font
@@
 			)
 		)
-		(property "Footprint" "Resistor_SMD:R_1206_3216Metric_Pad1.30x1.75mm_HandSolder"
+		(property "Footprint" "Resistor_SMD:R_0805_2012Metric_Pad1.20x1.40mm_HandSolder"
 			(at 222.758 130.81 90)
 			(effects
@@
 			)
 		)
-		(property "Footprint" "Capacitor_SMD:C_1206_3216Metric_Pad1.33x1.80mm_HandSolder"
+		(property "Footprint" "Capacitor_SMD:C_0805_2012Metric_Pad1.18x1.45mm_HandSolder"
 			(at 213.0552 133.985 0)
 			(effects
@@
 			)
 		)
-		(property "Footprint" "Resistor_SMD:R_1206_3216Metric_Pad1.30x1.75mm_HandSolder"
+		(property "Footprint" "Resistor_SMD:R_0805_2012Metric_Pad1.20x1.40mm_HandSolder"
 			(at 232.918 130.81 90)
 			(effects
@@
 	(symbol
 		(lib_id "Switch:SW_Push")
-		(at 43.18 67.945 0)
+		(at 43.18 65.405 0)
 		(unit 1)
 		(exclude_from_sim no)
@@
 		(fields_autoplaced yes)
 		(property "Reference" "SW2"
-			(at 43.18 60.325 0)
+			(at 43.18 57.15 0)
 			(effects
 				(font
@@
 			)
 		)
-		(property "Value" "SW_Push"
-			(at 43.18 62.865 0)
+		(property "Value" "UN/FOLD"
+			(at 43.18 59.69 0)
 			(effects
 				(font
@@
 		)
 		(property "Footprint" "Button_Switch_SMD:SW_SPST_PTS647_Sx38"
-			(at 43.18 62.865 0)
+			(at 43.18 60.325 0)
 			(effects
 				(font
@@
 		)
 		(property "Datasheet" "~"
-			(at 43.18 62.865 0)
+			(at 43.18 60.325 0)
 			(effects
 				(font
@@
 		)
 		(property "Description" "Push button switch, generic, two pins"
-			(at 43.18 67.945 0)
+			(at 43.18 65.405 0)
 			(effects
 				(font
@@
 		(on_board yes)
 		(dnp no)
-		(fields_autoplaced yes)
 		(property "Reference" "SW4"
-			(at 45.72 78.105 0)
+			(at 47.625 80.645 0)
 			(effects
 				(font
@@
 			)
 		)
-		(property "Value" "SW_Push"
-			(at 45.72 80.645 0)
+		(property "Value" "UP"
+			(at 47.625 82.55 0)
 			(effects
 				(font
@@
 		(on_board yes)
 		(dnp no)
-		(fields_autoplaced yes)
 		(property "Reference" "SW6"
-			(at 45.72 95.885 0)
+			(at 45.72 97.79 0)
 			(effects
 				(font
@@
 			)
 		)
-		(property "Value" "SW_Push"
-			(at 45.72 98.425 0)
+		(property "Value" "LEFT"
+			(at 45.72 99.695 0)
 			(effects
 				(font
@@
 			)
 		)
-		(property "Footprint" "Resistor_SMD:R_1206_3216Metric_Pad1.30x1.75mm_HandSolder"
+		(property "Footprint" "Resistor_SMD:R_0805_2012Metric_Pad1.20x1.40mm_HandSolder"
 			(at 180.213 132.08 90)
 			(effects
@@
 			)
 		)
-		(property "Footprint" "Package_TO_SOT_SMD:TO-252-3_TabPin2"
+		(property "Footprint" "Package_TO_SOT_SMD:TO-263-3_TabPin2"
 			(at 187.96 45.72 0)
 			(effects
@@
 		(on_board yes)
 		(dnp no)
-		(fields_autoplaced yes)
 		(property "Reference" "SW7"
-			(at 48.26 106.045 0)
+			(at 48.26 105.41 0)
 			(effects
 				(font
@@
 			)
 		)
-		(property "Value" "SW_Push"
-			(at 48.26 108.585 0)
+		(property "Value" "RIGHT"
+			(at 48.26 109.855 0)
 			(effects
 				(font
@@
 			)
 		)
-		(property "Footprint" "Resistor_SMD:R_1206_3216Metric_Pad1.30x1.75mm_HandSolder"
+		(property "Footprint" "Resistor_SMD:R_0805_2012Metric_Pad1.20x1.40mm_HandSolder"
 			(at 170.053 132.08 90)
 			(effects
@@
 		(on_board yes)
 		(dnp no)
-		(fields_autoplaced yes)
 		(property "Reference" "SW3"
-			(at 43.18 67.945 0)
+			(at 43.18 69.215 0)
 			(effects
 				(font
@@
 			)
 		)
-		(property "Value" "SW_Push"
-			(at 43.18 70.485 0)
+		(property "Value" "HEAT"
+			(at 43.18 71.12 0)
 			(effects
 				(font
@@
 		(on_board yes)
 		(dnp no)
-		(fields_autoplaced yes)
 		(property "Reference" "SW5"
-			(at 45.72 88.265 0)
+			(at 45.72 90.17 0)
 			(effects
 				(font
@@
 			)
 		)
-		(property "Value" "SW_Push"
-			(at 45.72 90.805 0)
+		(property "Value" "DOWN"
+			(at 45.72 92.075 0)
 			(effects
 				(font
@@
 			)
 		)
-		(property "Footprint" ""
+		(property "Footprint" "PracticasKiCad:LSF0002"
 			(at 190.5 139.7 0)
 			(effects

Commit message: .,.
Parts:
- removed R8: 0, Resistor_SMD:R_0805_2012Metric_Pad1.20x1.40mm_HandSolder, symbol Device:R
Connections:
- net GNDPWR is gone; now on net GND: C15.2, C16.2, C6.2, C8.2, D11.2 (A), D12.2 (A), D13.2 (A), D14.2 (A), J10.2 (Pin_2), J6.2 (Pin_2), J7.2 (Pin_2), R12.1, R17.1, R4.2, R5.2, U4.8 (GND)
- net SDA1: now reaches R11.2, U1.4 (SDA), U8.4 (B2)
- net OSC1: now reaches C12.1, U7.13 (OSC1/CLKI/RA7), Y1.1
- net OSC2: now reaches C13.1, U7.14 (OSC2/CLKO/RA6), Y1.2
- net OPA_N: now reaches R12.2, R15.1, U6.2 (-)
- net Tran_Int: now reaches D5.2 (A), Q2.3 (C), SW9.4
- net OPA_P: now reaches R13.1, R14.2, U6.3 (+)
- net FB: now reaches C18.1, R1.2, R2.1, U3.4 (FB)
- net SCL1: now reaches R10.2, U1.2 (SCL), U8.5 (B1)
- net Tran_Cal: now reaches D3.2 (A), Q3.3 (C), SW8.4
- net OPB_P: now reaches R16.2, R19.1, U6.5 (+)
- net OPB_N: now reaches R17.2, R18.1, U6.6 (-)
- net OUT_BUCK: now reaches D1.1 (K), L1.1, U3.2 (OUT)
Changed lines of the file:
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@@
 	(wire
 		(pts
-			(xy 205.74 189.865) (xy 210.82 189.865)
+			(xy 205.74 189.865) (xy 223.52 189.865)
 		)
 		(stroke
@@
 	(wire
 		(pts
-			(xy 218.44 189.865) (xy 223.52 189.865)
-		)
-		(stroke
-			(width 0)
-			(type default)
-		)
-	)
-	(wire
-		(pts
 			(xy 133.35 100.965) (xy 138.43 100.965)
 		)
@@
 		)
 	)
+	(label "OSC2"
+		(at 58.42 163.195 0)
+		(effects
+			(font
+				(size 1.27 1.27)
+			)
+			(justify left bottom)
+		)
+	)
 	(label "S_INT"
 		(at 227.33 140.97 180)
@@
 		)
 	)
+	(label "OSC1"
+		(at 60.325 160.655 0)
+		(effects
+			(font
+				(size 1.27 1.27)
+			)
+			(justify left bottom)
+		)
+	)
 	(label "Motor2B"
 		(at 375.285 87.63 0)
@@
 		)
 	)
+	(label "SDA1"
+		(at 208.28 148.59 0)
+		(effects
+			(font
+				(size 1.27 1.27)
+			)
+			(justify left bottom)
+		)
+	)
+	(label "OPA_P"
+		(at 314.96 177.165 90)
+		(effects
+			(font
+				(size 1.27 1.27)
+			)
+			(justify left bottom)
+		)
+	)
 	(label "Motor1B"
 		(at 339.725 55.88 0)
@@
 		)
 	)
+	(label "FB"
+		(at 144.78 33.655 0)
+		(effects
+			(font
+				(size 1.27 1.27)
+			)
+			(justify left bottom)
+		)
+	)
+	(label "OPA_N"
+		(at 314.96 189.23 90)
+		(effects
+			(font
+				(size 1.27 1.27)
+			)
+			(justify left bottom)
+		)
+	)
 	(label "S_PROG"
 		(at 159.385 165.735 0)
@@
 		)
 	)
+	(label "SCL1"
+		(at 207.645 144.78 0)
+		(effects
+			(font
+				(size 1.27 1.27)
+			)
+			(justify left bottom)
+		)
+	)
 	(label "M_D"
 		(at 361.315 81.28 0)
@@
 		)
 	)
+	(label "Tran_Int"
+		(at 202.565 248.92 0)
+		(effects
+			(font
+				(size 1.27 1.27)
+			)
+			(justify left bottom)
+		)
+	)
 	(label "S_PROG"
 		(at 228.6 152.4 180)
@@
 		)
 	)
+	(label "OPB_N"
+		(at 368.3 188.595 90)
+		(effects
+			(font
+				(size 1.27 1.27)
+			)
+			(justify left bottom)
+		)
+	)
+	(label "OUT_BUCK"
+		(at 136.525 45.72 0)
+		(effects
+			(font
+				(size 1.27 1.27)
+			)
+			(justify left bottom)
+		)
+	)
 	(label "S_SDA"
 		(at 149.225 147.955 0)
@@
 		)
 	)
+	(label "Tran_Cal"
+		(at 349.885 229.235 0)
+		(effects
+			(font
+				(size 1.27 1.27)
+			)
+			(justify left bottom)
+		)
+	)
 	(label "CAN-"
 		(at 76.2 261.62 0)
@@
 		)
 	)
+	(label "OPB_P"
+		(at 368.3 176.53 90)
+		(effects
+			(font
+				(size 1.27 1.27)
+			)
+			(justify left bottom)
+		)
+	)
 	(global_label "MCLR"
 		(shape input)
@@
 					(unit 1)
 				)
-			)
-		)
-	)
-	(symbol
-		(lib_id "Device:R")
-		(at 214.63 189.865 90)
-		(unit 1)
-		(exclude_from_sim no)
-		(in_bom yes)
-		(on_board yes)
-		(dnp no)
-		(property "Reference" "R8"
-			(at 214.63 192.405 90)
-			(effects
-				(font
-					(size 1.27 1.27)
-				)
-			)
-		)
-		(property "Value" "0"
-			(at 214.63 194.945 90)
-			(effects
-				(font
-					(size 1.27 1.27)
-				)
-			)
-		)
-		(property "Footprint" "Resistor_SMD:R_0805_2012Metric_Pad1.20x1.40mm_HandSolder"
-			(at 214.63 191.643 90)
-			(effects
-				(font
-					(size 1.27 1.27)
-				)
-				(hide yes)
-			)
-		)
-		(property "Datasheet" "~"
-			(at 214.63 189.865 0)
-			(effects
-				(font
-					(size 1.27 1.27)
-				)
-				(hide yes)
-			)
-		)
-		(property "Description" "Resistor"
-			(at 214.63 189.865 0)
-			(effects
-				(font
-					(size 1.27 1.27)
-				)
-				(hide yes)
-			)
-		)
-		(pin "1"
-		)
-		(pin "2"
-		)
-		(instances
-			(project ""
-				(path "/c3f67613-7195-4d14-ab28-355c40c698ae"
-					(reference "R8")
-					(unit 1)
-				)
