File: _autosave-DIMECRES_C_retrovisors.kicad_sch (KiCad schematic)
At the start: 41 parts, among them J1 Conn_Entrada, J2 DE9_Pins, J3 Conn_01x05_Pin, Q1 DTC144E, SW1 SW_DPDT_G6S, U1 PIC18F258-xSO, U2 LM1117DT-ADJ, U3 LM2596S-ADJ, U4 L298N, U5 TJA1042T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

Commit message: Upload sch
Parts:
- added C12, C13: 15p, Capacitor_SMD:C_0805_2012Metric_Pad1.18x1.45mm_HandSolder, symbol Device:C
- added C14: 100n, symbol Device:C
- added J4: Botonera, symbol Connector:Conn_01x06_Pin
- added U7: PIC18F4480-IP, Package_DIP:DIP-40_W15.24mm, symbol MCU_Microchip_PIC18:PIC18F4480-IP
- added Y1: Crystal, PracticasKiCad:Crystal_SMD_HC49-SD_Practica3, symbol Device:Crystal
Connections:
- net Act_Rele_M2/M3: no longer U1.11 (RC0/SOSCO)
- net ENA: now also U7.17 (CCP1/RC2); no longer U1.23 (RB2)
- net ENB: now also U7.24 (SDO/RC5); no longer U1.26 (RB5)
- net FiCa_A: now also U7.2 (RA0/AN0/CVref); no longer U1.3 (RA1)
- net FiCa_B: now also U7.3 (RA1/AN1); no longer U1.4 (RA2)
- net GND: now also C12.2, C13.2, C14.2, U7.12 (VSS), U7.31 (VSS); no longer U1.19 (VSS), U1.8 (VSS)
- net IN1A: now also U7.15 (T13CKI/T1OSO/RC0); no longer U1.21 (RB0)
- net IN1B: now also U7.16 (T1OSI/RC1); no longer U1.22 (RB1)
- net IN2/3A: now also U7.18 (SCL/SCK/RC3); no longer U1.24 (RB3)
- net IN2/3B: now also U7.23 (SDA/SDI/RC4); no longer U1.25 (RB4)
- net MCLR: now also U7.1 (~{MCLR}/VPP/RE3); no longer U1.1 (~{MCLR}/VPP/RE3)
- net PGC: now also U7.39 (RB6/KBI2/PGC); no longer U1.27 (RB6/PGC)
- net PGD: now also U7.40 (RB7/KBI3/PGD); no longer U1.28 (RB7/PGD)
- net Vcc: now also C14.1, U7.11 (VDD), U7.32 (VDD); no longer U1.20 (VDD)
- net RXCAN: no longer names the net of U1.17 (RC6)
- net RXCAN: no longer U5.4 (RXD)
- net TXCAN: no longer names the net of U1.18 (RC7)
- net TXCAN: no longer U5.1 (TXD)
- new net CANRX: U5.1 (TXD), U7.36 (RB3/CANRX)
- new net CANTX: U5.4 (RXD), U7.35 (RB2/INT2/CANTX)
- new net XTAL1: C12.1, U7.13 (OSC1/CLKI/RA7), Y1.1
- new net XTAL2: C13.1, U7.14 (OSC2/CLKO/RA6), Y1.2
Other:
- note added: "OSCILLATOR CIRCUIT"
- moved on the sheet: C9, U1
