File: DIMECRES_C_retrovisors.kicad_pcb (KiCad board)
At the start: 2 copper layers, 79 parts, among them J10 Vbat, J2 DE9_Pins, J3 Conn_01x05_Pin, J4 Motor3, J5 DE9_Pins, J6 Intermitente, J7 Calentador, J8 Motor2, J9 Motor1, Q1 DTC144E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

Commit message: Inicio Layout queda mucho aun...
Parts:
- C7, C8: moved to B.Cu
- R4, R5: footprint Resistor_SMD:R_Shunt_Vishay_WSR2_WSR3 -> Resistor_SMD:R_1206_3216Metric_Pad1.30x1.75mm_HandSolder
- moved SW1 205.9 mm to (68.0, 75.7)
- moved J5 201.6 mm to (207.7, 275.9)
- moved J6 201.6 mm to (251.1, 261.0)
- moved J7 201.6 mm to (251.7, 249.0)
- moved R4 190.0 mm to (78.9, 57.9), turned to 90 degrees
- moved C17 188.7 mm to (74.6, 67.8), turned to 90 degrees
- moved R5 183.5 mm to (80.5, 86.2)
- moved Q1 182.8 mm to (70.2, 53.8), turned to 180 degrees
- moved D1 182.1 mm to (72.3, 134.7)
- moved U6 178.4 mm to (91.8, 39.6)
- moved C8 175.4 mm to (81.8, 65.8), turned to 90 degrees
- moved C7 175.0 mm to (81.1, 75.3), turned to -90 degrees
- moved C4 174.5 mm to (89.3, 128.2), turned to -90 degrees
- moved D6 167.7 mm to (72.0, 64.6), turned to 180 degrees
- moved R21 164.1 mm to (108.0, 134.5), turned to 180 degrees
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Connections:
- net /Motor1+ renamed /Motor1A
- net /Motor1- renamed /Motor1B
- net /Motor2+ renamed /Motor2A
- net /Motor23+ renamed /Motor23A
- net /Motor23- renamed /Motor23B
- net /Motor3+ renamed /Motor3A
- net Net-(D6-A) renamed /M_D
- net Net-(U10-VI) renamed /V_6
- J4 pad 2: /Motor2- -> /Motor3B
- J8 pad 2: /Motor2- -> /Motor2B
- SW1 pad 3: /Motor2- -> /Motor2B
- SW1 pad 5: /Motor2- -> /Motor3B
- U7 pad 10: unconnected-(U7-C2OUT/AN7/~{CS}/RE2-Pad10) -> Act_Rele_M2/M3
- U7 pad 22: unconnected-(U7-C2IN-/PSP3/RD3-Pad22) -> B_Down
- U7 pad 24: Calentador -> /S_PROG
- U7 pad 27: B_Un/Fold -> B_Left
- U7 pad 28: B_Heat -> B_Right
- U7 pad 29: /S_PROG -> B_Up
- U7 pad 30: /S_INT -> B_Heat
- U7 pad 33: Act_Rele_M2/M3 -> B_Un/Fold
- U7 pad 34: unconnected-(U7-RB1/INT1/AN8-Pad34) -> /S_INT
- U7 pad 38: unconnected-(U7-RB5/KBI1/PGM-Pad38) -> Calentador
- U7 pad 4: B_Up -> unconnected-(U7-RA2/AN2/Vref--Pad4)
- U7 pad 5: B_Down -> unconnected-(U7-RA3/AN3/Vref+-Pad5)
- U7 pad 6: B_Left -> unconnected-(U7-RA4/TOCKI-Pad6)
- U7 pad 7: B_Right -> unconnected-(U7-RA5/ANA4/~{SS}/HLVDIN-Pad7)
Routing:
- net EN2/3: track 0.00 -> 49.0 mm
- net /S_INT: track 0.00 -> 44.6 mm, vias 0 -> 2
- net Act_Rele_M2/M3: track 0.00 -> 42.5 mm
- net Vbat: track 0.00 -> 36.2 mm
- net /S_SCL: track 0.00 -> 35.5 mm
- net IN1A: track 0.00 -> 35.3 mm
- net IN1B: track 0.00 -> 33.8 mm
- net /Motor1A: track 0.00 -> 33.4 mm
- net B_Heat: track 0.00 -> 30.5 mm
- net /Motor1B: track 0.00 -> 29.6 mm
- net B_Right: track 0.00 -> 29.2 mm
- net IN2/3B: track 0.00 -> 27.2 mm
- net IN2/3A: track 0.00 -> 27.2 mm
- net EN1: track 0.00 -> 27.2 mm
- net B_Down: track 0.00 -> 27.1 mm
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- added copper zone on B.Cu, net GND
- added copper zone on F.Cu, net Vcc

Commit message: Todo el layout v1 ?
Parts:
- removed C6: 47n, Capacitor_SMD:C_1206_3216Metric_Pad1.33x1.80mm_HandSolder
- removed R6, R7: 60, Resistor_SMD:R_0805_2012Metric_Pad1.20x1.40mm_HandSolder
- added JP1: Jumper_3_Open, Connector_PinHeader_2.54mm:PinHeader_1x03_P2.54mm_Vertical, F.Cu at (128.5, 115.4)
- added R9: 33k, LED_SMD:LED_1206_3216Metric_Pad1.42x1.75mm_HandSolder, F.Cu at (134.1, 114.8)
- added SW10: SW_Push, Button_Switch_SMD:SW_SPST_PTS647_Sx38, F.Cu at (134.2, 119.9)
- C10, C11, C14, C15, C16, C20, C21, C22, C9: moved to B.Cu
- moved J5 236.4 mm to (116.4, 57.8), turned to 180 degrees
- moved J6 185.7 mm to (179.0, 89.9), turned to 90 degrees
- moved C19 166.1 mm to (102.1, 63.9), turned to -90 degrees
- moved J7 164.3 mm to (179.0, 101.6), turned to 90 degrees
- moved C20 163.2 mm to (105.2, 64.4), turned to -90 degrees
- moved C3 160.6 mm to (95.6, 64.0), turned to -90 degrees
- moved C10 155.6 mm to (111.0, 110.8)
- moved C14 143.7 mm to (118.6, 90.0), turned to 90 degrees
- moved J2 134.7 mm to (100.0, 118.1), turned to -90 degrees
- moved J4 130.4 mm to (179.1, 54.9), turned to 90 degrees
- moved J9 128.1 mm to (179.0, 77.5), turned to 90 degrees
- moved J8 127.3 mm to (179.1, 66.3), turned to 90 degrees
- moved C9 127.1 mm to (129.0, 84.8), turned to 90 degrees
- moved C11 126.9 mm to (136.6, 96.0)
- moved J10 114.6 mm to (178.9, 113.2), turned to 90 degrees
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Connections:
- J3 pad 1: MCLR -> /prog
- U7 pad 22: B_Down -> B_Up
- U7 pad 27: B_Left -> B_Right
- U7 pad 28: B_Right -> B_Left
- U7 pad 29: B_Up -> B_Down
- U7 pad 38: Calentador -> unconnected-(U7-RB5/KBI1/PGM-Pad38)
- U7 pad 4: unconnected-(U7-RA2/AN2/Vref--Pad4) -> AngleMort
- U7 pad 5: unconnected-(U7-RA3/AN3/Vref+-Pad5) -> Calentador
- U7 pad 8: AngleMort -> unconnected-(U7-AN5/~{RD}/RE0-Pad8)
Routing:
- net Vbat: track 36.2 -> 120.0 mm, vias 0 -> 1
- net AngleMort: track 0.00 -> 43.0 mm, vias 0 -> 1
- net SENSE_B: track 10.1 -> 42.7 mm
- net Vdd: track 0.00 -> 27.9 mm
- net Net-(D5-A): track 0.00 -> 21.3 mm
- net MAN_MCLR: track 0.00 -> 20.9 mm
- net Tx: track 0.00 -> 20.6 mm
- net Intermitente: track 0.00 -> 20.0 mm, vias 0 -> 2
- net Calentador: track 0.00 -> 18.7 mm, vias 0 -> 1
- net Rx: track 0.00 -> 16.9 mm
- net Net-(J6-Pin_1): track 0.00 -> 16.6 mm
- net Net-(J7-Pin_1): track 0.00 -> 15.9 mm
- net B_Right: track 29.2 -> 13.5 mm
- net B_Left: track 13.5 -> 29.2 mm
- net /CAN+: track 0.00 -> 15.3 mm
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- added copper zone on F.Cu, net GND
- added copper zone on B.Cu, net GNDPWR
- added copper zone on F.Cu, net Vbat
Other:
- board outline added: 97.2 x 83.4 mm

Commit message: -|-
Parts:
- R8: moved to B.Cu
- moved R8 40.3 mm to (182.6, 116.8), turned to 90 degrees
Changed lines of the file:
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@@
 		)
 	)
-	(footprint "Resistor_SMD:R_0805_2012Metric_Pad1.20x1.40mm_HandSolder"
-		(layer "F.Cu")
-		(at 200.4 80.6)
-		(descr "Resistor SMD 0805 (2012 Metric), square (rectangular) end terminal, IPC_7351 nominal with elongated pad for handsoldering. (Body size source: IPC-SM-782 page 72, https://www.pcb-3d.com/wordpress/wp-content/uploads/ipc-sm-782a_amendment_1_and_2.pdf), generated with kicad-footprint-generator")
-		(tags "resistor handsolder")
-		(property "Reference" "R8"
-			(at 0 -1.65 0)
-			(layer "F.SilkS")
-			(effects
-				(font
-					(size 1 1)
-					(thickness 0.15)
-				)
-			)
-		)
-		(property "Value" "0"
-			(at 0 1.65 0)
-			(layer "F.Fab")
-			(effects
-				(font
-					(size 1 1)
-					(thickness 0.15)
-				)
-			)
-		)
-		(property "Datasheet" ""
-			(at 0 0 0)
-			(unlocked yes)
-			(layer "F.Fab")
-			(hide yes)
-			(effects
-				(font
-					(size 1.27 1.27)
-					(thickness 0.15)
-				)
-			)
-		)
-		(property "Description" "Resistor"
-			(at 0 0 0)
-			(unlocked yes)
-			(layer "F.Fab")
-			(hide yes)
-			(effects
-				(font
-					(size 1.27 1.27)
-					(thickness 0.15)
-				)
-			)
-		)
-		(property ki_fp_filters "R_*")
-		(sheetname "/")
-		(sheetfile "DIMECRES_C_retrovisors.kicad_sch")
-		(attr smd)
-		(fp_line
-			(start -0.227064 -0.735)
-			(end 0.227064 -0.735)
-			(stroke
-				(width 0.12)
-				(type solid)
-			)
-			(layer "F.SilkS")
-		)
-		(fp_line
-			(start -0.227064 0.735)
-			(end 0.227064 0.735)
-			(stroke
-				(width 0.12)
-				(type solid)
-			)
-			(layer "F.SilkS")
-		)
-		(fp_line
-			(start -1.85 -0.95)
-			(end 1.85 -0.95)
-			(stroke
-				(width 0.05)
-				(type solid)
-			)
-			(layer "F.CrtYd")
-		)
-		(fp_line
-			(start -1.85 0.95)
-			(end -1.85 -0.95)
-			(stroke
-				(width 0.05)
-				(type solid)
-			)
-			(layer "F.CrtYd")
-		)
-		(fp_line
-			(start 1.85 -0.95)
-			(end 1.85 0.95)
-			(stroke
-				(width 0.05)
-				(type solid)
-			)
-			(layer "F.CrtYd")
-		)
-		(fp_line
-			(start 1.85 0.95)
-			(end -1.85 0.95)
-			(stroke
-				(width 0.05)
-				(type solid)
-			)
-			(layer "F.CrtYd")
-		)
-		(fp_line
-			(start -1 -0.625)
-			(end 1 -0.625)
-			(stroke
-				(width 0.1)
-				(type solid)
-			)
-			(layer "F.Fab")
-		)
-		(fp_line
-			(start -1 0.625)
-			(end -1 -0.625)
-			(stroke
-				(width 0.1)
-				(type solid)
-			)
-			(layer "F.Fab")
-		)
-		(fp_line
-			(start 1 -0.625)
-			(end 1 0.625)
-			(stroke
-				(width 0.1)
-				(type solid)
-			)
-			(layer "F.Fab")
-		)
-		(fp_line
-			(start 1 0.625)
-			(end -1 0.625)
-			(stroke
-				(width 0.1)
-				(type solid)
-			)
-			(layer "F.Fab")
-		)
-		(fp_text user "${REFERENCE}"
-			(at 0 0 0)
-			(layer "F.Fab")
-			(effects
-				(font
-					(size 0.5 0.5)
-					(thickness 0.08)
-				)
-			)
-		)
-		(pad "1" smd roundrect
-			(at -1 0)
-			(size 1.2 1.4)
-			(layers "F.Cu" "F.Mask" "F.Paste")
-			(roundrect_rratio 0.208333)
-			(net 1 "GND")
-			(pintype "passive")
-		)
-		(pad "2" smd roundrect
-			(at 1 0)
-			(size 1.2 1.4)
-			(layers "F.Cu" "F.Mask" "F.Paste")
-			(roundrect_rratio 0.208333)
-			(net 6 "GNDPWR")
-			(pintype "passive")
-		)
-		(embedded_fonts no)
-		(model "${KICAD9_3DMODEL_DIR}/Resistor_SMD.3dshapes/R_0805_2012Metric.wrl"
-			(offset
-				(xyz 0 0 0)
-			)
-			(scale
-				(xyz 1 1 1)
-			)
-			(rotate
-				(xyz 0 0 0)
-			)
-		)
-	)
 	(footprint "Resistor_SMD:R_1206_3216Metric_Pad1.30x1.75mm_HandSolder"
 		(layer "F.Cu")
@@
 			(offset
 				(xyz 0 0 0)
+			)
+			(scale
+				(xyz 1 1 1)
+			)
+			(rotate
+				(xyz 0 0 0)
+			)
+		)
+	)
+	(footprint "Resistor_SMD:R_0805_2012Metric_Pad1.20x1.40mm_HandSolder"
+		(layer "B.Cu")
+		(at 182.6 116.8 90)
+		(descr "Resistor SMD 0805 (2012 Metric), square (rectangular) end terminal, IPC_7351 nominal with elongated pad for handsoldering. (Body size source: IPC-SM-782 page 72, https://www.pcb-3d.com/wordpress/wp-content/uploads/ipc-sm-782a_amendment_1_and_2.pdf), generated with kicad-footprint-generator")
+		(tags "resistor handsolder")
+		(property "Reference" "R8"
+			(at 0 1.65 90)
+			(layer "B.SilkS")
+			(effects
+				(font
+					(size 1 1)
+					(thickness 0.15)
+				)
+				(justify mirror)
+			)
+		)
+		(property "Value" "0"
+			(at 0 -1.65 90)
+			(layer "B.Fab")
+			(effects
+				(font
+					(size 1 1)
+					(thickness 0.15)
+				)
+				(justify mirror)
+			)
+		)
+		(property "Datasheet" ""
+			(at 0 0 270)
+			(unlocked yes)
+			(layer "B.Fab")
+			(hide yes)
+			(effects
+				(font
+					(size 1.27 1.27)
+					(thickness 0.15)
+				)
+				(justify mirror)
+			)
+		)
+		(property "Description" "Resistor"
+			(at 0 0 270)
+			(unlocked yes)
+			(layer "B.Fab")
+			(hide yes)
+			(effects
+				(font
+					(size 1.27 1.27)
+					(thickness 0.15)
+				)
+				(justify mirror)
+			)
+		)
+		(property ki_fp_filters "R_*")
+		(sheetname "/")
+		(sheetfile "DIMECRES_C_retrovisors.kicad_sch")
+		(attr smd)
+		(fp_line
+			(start -0.227064 -0.735)
+			(end 0.227064 -0.735)
+			(stroke
+				(width 0.12)
+				(type solid)
+			)
+			(layer "B.SilkS")
+		)
+		(fp_line
+			(start -0.227064 0.735)
+			(end 0.227064 0.735)
+			(stroke
+				(width 0.12)
+				(type solid)
+			)
+			(layer "B.SilkS")
+		)
+		(fp_line
+			(start 1.85 -0.95)
+			(end -1.85 -0.95)
+			(stroke
+				(width 0.05)
+				(type solid)
+			)
+			(layer "B.CrtYd")
+		)
+		(fp_line
+			(start -1.85 -0.95)
+			(end -1.85 0.95)
+			(stroke
+				(width 0.05)
+				(type solid)
+			)
+			(layer "B.CrtYd")
+		)
+		(fp_line
+			(start 1.85 0.95)
+			(end 1.85 -0.95)
+			(stroke
+				(width 0.05)
+				(type solid)
+			)
+			(layer "B.CrtYd")
+		)
+		(fp_line
+			(start -1.85 0.95)
+			(end 1.85 0.95)
+			(stroke
+				(width 0.05)
+				(type solid)
+			)
+			(layer "B.CrtYd")
+		)
+		(fp_line
+			(start 1 -0.625)
+			(end -1 -0.625)
+			(stroke
+				(width 0.1)
+				(type solid)
+			)
+			(layer "B.Fab")
+		)
+		(fp_line
+			(start -1 -0.625)
+			(end -1 0.625)
+			(stroke
+				(width 0.1)
+				(type solid)
+			)
+			(layer "B.Fab")
+		)
+		(fp_line
+			(start 1 0.625)
+			(end 1 -0.625)
+			(stroke
+				(width 0.1)
+				(type solid)
+			)
+			(layer "B.Fab")
+		)
+		(fp_line
+			(start -1 0.625)
+			(end 1 0.625)
+			(stroke
+				(width 0.1)
+				(type solid)
+			)
+			(layer "B.Fab")
+		)
+		(fp_text user "${REFERENCE}"
+			(at 0 0 90)
+			(layer "B.Fab")
+			(effects
+				(font
+					(size 0.5 0.5)
+					(thickness 0.08)
+				)
+				(justify mirror)
+			)
+		)
+		(pad "1" smd roundrect
+			(at -1 0 90)
+			(size 1.2 1.4)
+			(layers "B.Cu" "B.Mask" "B.Paste")
+			(roundrect_rratio 0.208333)
+			(net 1 "GND")
+			(pintype "passive")
+		)
+		(pad "2" smd roundrect
+			(at 1 0 90)
+			(size 1.2 1.4)
+			(layers "B.Cu" "B.Mask" "B.Paste")
+			(roundrect_rratio 0.208333)
+			(net 6 "GNDPWR")
+			(pintype "passive")
+		)
+		(embedded_fonts no)
+		(model "${KICAD9_3DMODEL_DIR}/Resistor_SMD.3dshapes/R_0805_2012Metric.wrl"
+			(offset
+				(xyz 0 0 0)

Commit message: Actu Layoutt
Parts:
- added C6: 47n, Capacitor_SMD:C_1206_3216Metric_Pad1.33x1.80mm_HandSolder, F.Cu at (108.2, 117.2)
- added REF**: MountingHole_3.2mm_M3, MountingHole:MountingHole_3.2mm_M3, F.Cu at (92.4, 49.0)
- added REF**: MountingHole_3.2mm_M3, MountingHole:MountingHole_3.2mm_M3, F.Cu at (95.8, 124.8)
- added REF**: MountingHole_3.2mm_M3, MountingHole:MountingHole_3.2mm_M3, F.Cu at (181.5, 49.3)
- added REF**: MountingHole_3.2mm_M3, MountingHole:MountingHole_3.2mm_M3, F.Cu at (181.3, 124.9)
- C20: moved to F.Cu
- moved J4 16.0 mm to (163.8, 50.2), turned to 0 degrees
- moved C20 6.38 mm to (102.1, 58.8), turned to 90 degrees
- moved J6 5.04 mm to (179.0, 84.8), turned to -90 degrees
- moved Q1 5.02 mm to (162.6, 84.2)
- moved J10 5.02 mm to (179.1, 108.2), turned to -90 degrees
- moved J7 5.01 mm to (179.0, 96.6), turned to -90 degrees
- moved J9 4.93 mm to (179.1, 72.6), turned to -90 degrees
- moved J8 4.80 mm to (179.1, 61.5), turned to -90 degrees
- moved SW3 4.54 mm to (94.8, 93.8)
- moved SW2 2.98 mm to (107.9, 93.5)
- moved SW5 2.98 mm to (100.9, 86.2)
- moved SW6 2.95 mm to (93.6, 80.7)
- moved SW4 2.94 mm to (100.9, 75.2)
- moved SW7 2.88 mm to (108.2, 80.7)
- moved R5 2.28 mm to (157.2, 83.0)
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Connections:
- net Net-(J6-Pin_1) renamed /M_Inter
- net Net-(J7-Pin_1) renamed /M_calen
Routing:
- net GND: track 0.00 -> 102.3 mm, vias 0 -> 69
- net Vcc: track 0.00 -> 28.6 mm, vias 0 -> 4
- net Vbat: track 120.0 -> 103.9 mm, vias 1 -> 6
- net CANTX: track 0.00 -> 12.9 mm
- net /Motor1B: track 29.6 -> 42.2 mm
- net /Motor3A: track 22.8 -> 12.0 mm
- net GNDPWR: track 0.00 -> 9.38 mm, vias 0 -> 8
- net CANRX: track 0.00 -> 8.78 mm
- net /Motor3B: track 16.0 -> 9.77 mm
- net B_Left: track 29.2 -> 26.0 mm
- net Act_Rele_M2/M3: track 36.1 -> 33.0 mm
- net B_Un/Fold: track 14.8 -> 11.7 mm
- net B_Heat: track 29.7 -> 26.6 mm
- net /M_D: track 15.7 -> 18.6 mm
- net B_Down: track 21.0 -> 18.4 mm
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Other:
- board size 97.2 x 83.4 mm -> 96.2 x 83.4 mm
- board text added: "GND"
- board text added: "PGC"
- board text added: "PGD"
- board text added: "PRG"
- board text added: "Vcc"

Commit message: .,.,-
Parts:
- removed C6: 47n, Capacitor_SMD:C_1206_3216Metric_Pad1.33x1.80mm_HandSolder
- added R7: 15k, Resistor_SMD:R_1206_3216Metric_Pad1.30x1.75mm_HandSolder, F.Cu at (111.7, 117.2)
- U5: value TJA1042T -> MCP2551-I-SN
- moved D4 101.8 mm to (99.3, 49.1)
- moved R21 101.8 mm to (103.7, 49.0)
- moved R20 28.4 mm to (140.5, 120.8)
- moved D2 28.4 mm to (144.7, 120.8)
- moved J9 5.18 mm to (179.1, 77.8), turned to 90 degrees
- moved U3 0.13 mm to (159.9, 119.2)
- moved U5 0.13 mm to (110.2, 110.9)
Connections:
- C22 pad 1: Vbat -> Vcc
- C22 pad 2: GNDPWR -> GND
- D3 pad 1: Vbat -> Vcc
- SW8 pad 3: Vbat -> Vcc
- U5 pad 5: Net-(U5-SPLIT) -> unconnected-(U5-Vref-Pad5)
- U5 pad 8: GND -> Net-(U5-Rs)
Routing:
- net Vbat: track 103.9 -> 12.3 mm, vias 6 -> 5
- net GND: track 102.3 -> 55.3 mm, vias 69 -> 76
- net AngleMort: track 43.0 -> 24.6 mm, vias 1 -> 0
- net /Motor1B: track 42.2 -> 30.1 mm
- net Net-(U5-Rs): track 0.00 -> 3.01 mm
- net Net-(U5-SPLIT): track 2.36 -> 0.00 mm
- net /Motor1A: track 35.5 -> 33.6 mm
Other:
- board size 96.2 x 83.4 mm -> 97.6 x 83.4 mm

Commit message: Primeres MOdificacions Layout
Parts:
- added R22: 120, Resistor_SMD:R_0805_2012Metric_Pad1.20x1.40mm_HandSolder, F.Cu at (147.8, 102.6)
- added R23: 120, Resistor_SMD:R_0805_2012Metric_Pad1.20x1.40mm_HandSolder, F.Cu at (149.6, 95.8)
- added R24: 180, Resistor_SMD:R_0805_2012Metric_Pad1.20x1.40mm_HandSolder, F.Cu at (150.6, 68.3)
- moved C7 24.0 mm to (165.1, 82.0), turned to -90 degrees
- moved Q1 19.8 mm to (152.9, 66.9)
- moved D6 17.7 mm to (155.8, 56.8), turned to -90 degrees
- moved C17 16.3 mm to (159.3, 54.9), turned to 90 degrees
- moved C8 8.13 mm to (157.2, 71.1), turned to 180 degrees
- moved R14 7.07 mm to (147.6, 90.0), turned to -90 degrees
- moved C21 6.47 mm to (158.2, 86.1), turned to 180 degrees
- moved C22 5.33 mm to (159.1, 98.7), turned to 180 degrees
- moved J9 5.11 mm to (179.1, 72.7), turned to -90 degrees
- moved R4 4.50 mm to (158.8, 83.0)
- moved U4 4.36 mm to (155.0, 78.5), turned to 0 degrees
- moved R16 3.86 mm to (144.7, 90.0), turned to -90 degrees
- moved C15 3.49 mm to (164.3, 93.2)
- moved SW1 2.78 mm to (165.8, 62.9), turned to 90 degrees
- moved R8 2.72 mm to (185.2, 117.7)
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Connections:
- C17 pad 1: Vbat -> Vcc
- C17 pad 2: GNDPWR -> GND
- C21 pad 1: Vbat -> Vcc
- C21 pad 2: GNDPWR -> GND
- D5 pad 1: Vbat -> Vcc
- D6 pad 1: Vbat -> Vcc
- Q1 pad 2: GND -> Net-(Q1-E)
- Q2 pad 2: GND -> Net-(Q2-E)
- Q3 pad 2: GND -> Net-(Q3-E)
- SW1 pad 12: Vbat -> Vcc
- SW9 pad 3: Vbat -> Vcc
Routing:
- net Vcc: track 28.6 -> 60.9 mm, vias 4 -> 7
- net IN2/3B: track 16.4 -> 42.7 mm
- net IN2/3A: track 16.4 -> 41.3 mm
- net EN1: track 16.4 -> 39.8 mm
- net EN2/3: track 38.3 -> 58.0 mm, vias 0 -> 6
- net IN1B: track 26.4 -> 42.9 mm, vias 0 -> 4
- net /Motor23A: track 7.62 -> 23.3 mm
- net /Motor23B: track 23.5 -> 8.41 mm
- net IN1A: track 25.3 -> 38.0 mm, vias 0 -> 2
- net /M_D: track 18.6 -> 5.97 mm, vias 1 -> 0
- net Net-(D5-A): track 21.7 -> 9.15 mm
- net SENSE_B: track 44.5 -> 33.3 mm, vias 1 -> 0
- net Act_Rele_M2/M3: track 33.0 -> 43.5 mm, vias 2 -> 0
- net /Motor3B: track 9.77 -> 19.8 mm
- net /Motor1A: track 33.6 -> 24.6 mm, vias 0 -> 2
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Other:
- board size 97.6 x 83.4 mm -> 97.6 x 85 mm

Commit message: mod. lay.
Parts:
- SW2: value SW_Push -> UN/FOLD
- SW3: value SW_Push -> HEAT
- moved SW6 4.25 mm to (97.8, 80.8)
- moved R21 3.15 mm to (106.9, 48.9)
- moved D4 3.15 mm to (102.5, 49.0)
- moved J5 2.60 mm to (116.9, 55.9)
- moved REF** 2.55 mm to (94.5, 47.5)
- moved REF** 2.53 mm to (183.2, 47.4)
- moved SW3 2.49 mm to (97.2, 93.3)
- moved SW4 2.35 mm to (103.3, 75.3)
- moved SW5 2.30 mm to (103.2, 86.2)
- moved REF** 2.06 mm to (183.2, 125.5)
- moved J2 1.75 mm to (102.3, 118.5)
- moved R22 1.71 mm to (146.7, 101.3)
- moved SW2 1.70 mm to (109.6, 93.5)
- moved REF** 1.19 mm to (97.0, 125.0)
- moved C21 0.72 mm to (159.0, 86.0)
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Routing:
- net Net-(D5-A): track 9.15 -> 21.1 mm
- net B_Left: track 26.0 -> 21.7 mm
- net Vcc: track 60.9 -> 64.4 mm
- net Act_Rele_M2/M3: track 43.5 -> 40.3 mm
- net Tx: track 20.8 -> 23.5 mm
- net Rx: track 16.2 -> 18.9 mm
- net Net-(D1-K): track 16.5 -> 19.2 mm
- net B_Heat: track 26.6 -> 24.0 mm
- net B_Down: track 18.4 -> 15.9 mm
- net B_Up: track 24.5 -> 22.2 mm
- net /CAN+: track 15.0 -> 13.1 mm
- net /CAN-: track 14.9 -> 13.1 mm
- net B_Un/Fold: track 11.7 -> 9.95 mm
- net Net-(Q1-E): track 0.00 -> 1.66 mm
- net /S_PROG: track 15.7 -> 14.3 mm
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Other:
- board size 97.6 x 85 mm -> 96.5 x 85 mm

Commit message: Modificacions Layout
Parts:
- SW4: value SW_Push -> UP
- SW5: value SW_Push -> DOWN
- SW6: value SW_Push -> LEFT
- SW7: value SW_Push -> RIGHT
Routing:
- net GND: track 52.3 -> 57.2 mm, vias 75 -> 77
- net MAN_MCLR: track 18.5 -> 19.9 mm
- net MCLR: track 7.12 -> 8.49 mm
- net Net-(D1-K): track 19.2 -> 20.5 mm
