File: DIMECRES_C_retrovisors.kicad_pcb (KiCad board)
At the start: 2 copper layers, 96.5 x 85 mm, 87 parts, among them J10 Vbat, J2 DE9_Pins, J3 Conn_01x05_Pin, J4 Motor3, J5 DE9_Pins, J6 Intermitente, J7 Calentador, J8 Motor2, J9 Motor1, Q1 DTC144E, Q2 DTC144E, Q3 DTC144E, SW1 SW_DPDT_G6S, SW10 SW_Push, SW2 UN/FOLD, SW3 HEAT, SW4 UP, SW5 DOWN, SW6 LEFT, SW7 RIGHT, SW8 FN01B, SW9 FN01B, U1 CH201, U10 LM1117DT-5.0, U2 ADM7160, U3 LM2596S-ADJ, U4 L298N, U5 MCP2551-I-SN, U6 ADA4511-2, U7 PIC18F4480-IP, Y1 Crystal

Commit message: Proimeres correccions
Parts:
- removed C7: 100n, Capacitor_SMD:C_1206_3216Metric_Pad1.33x1.80mm_HandSolder
- added C6: 470U, Capacitor_THT:CP_Radial_D6.3mm_P2.50mm, F.Cu at (166.8, 88.7)
- added D10: 1N5822, Diode_THT:D_DO-201AD_P15.24mm_Horizontal, F.Cu at (143.6, 80.0)
- added D11: 1N5822, Diode_THT:D_DO-201AD_P15.24mm_Horizontal, F.Cu at (174.5, 91.8)
- added D12: 1N5822, Diode_THT:D_DO-201AD_P15.24mm_Horizontal, F.Cu at (173.0, 97.5)
- added D13: 1N5822, Diode_THT:D_DO-201AD_P15.24mm_Horizontal, F.Cu at (160.4, 97.6)
- added D14: 1N5822, Diode_THT:D_DO-201AD_P15.24mm_Horizontal, F.Cu at (158.9, 91.7)
- added D7: 1N5822, Diode_THT:D_DO-201AD_P15.24mm_Horizontal, F.Cu at (189.7, 80.3)
- added D8: 1N5822, Diode_THT:D_DO-201AD_P15.24mm_Horizontal, F.Cu at (188.3, 86.0)
- added D9: 1N5822, Diode_THT:D_DO-201AD_P15.24mm_Horizontal, F.Cu at (145.2, 85.9)
- added R6: 60, Resistor_SMD:R_0805_2012Metric_Pad1.20x1.40mm_HandSolder, F.Cu at (168.7, 332.7)
- C8: moved to F.Cu
- SW2: value UN/FOLD -> SW_Push
- SW3: value HEAT -> SW_Push
- SW4: value UP -> SW_Push
- SW5: value DOWN -> SW_Push
- SW6: value LEFT -> SW_Push
- SW7: value RIGHT -> SW_Push
- moved R8 231.1 mm to (-40.0, 170.1)
- moved D3 195.1 mm to (89.9, 275.5)
- moved R23 195.1 mm to (84.7, 279.7)
- moved C11 195.1 mm to (71.7, 280.6)
- moved C14 195.1 mm to (53.7, 273.9)
- moved Q3 195.1 mm to (84.8, 284.5)
- moved SW9 195.1 mm to (93.1, 272.1)
- moved C15 195.1 mm to (99.4, 277.2)
- moved C16 195.1 mm to (99.5, 282.7)
- moved C17 195.1 mm to (94.3, 238.8)
- moved C19 195.1 mm to (37.2, 247.8)
- moved C20 195.1 mm to (37.1, 242.8)
- moved C21 195.1 mm to (94.0, 270.0)
- moved C22 195.1 mm to (94.1, 282.6)
- moved C3 195.1 mm to (30.7, 247.9)
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Connections:
- U7 pad 10: Act_Rele_M2/M3 -> IN2/3B
- U7 pad 15: IN1A -> unconnected-(U7-T13CKI/T1OSO/RC0-Pad15)
- U7 pad 16: IN1B -> unconnected-(U7-T1OSI/RC1-Pad16)
- U7 pad 17: EN1 -> Act_Rele_M2/M3
- U7 pad 19: IN2/3A -> unconnected-(U7-C1IN+/PSP0/RD0-Pad19)
- U7 pad 20: IN2/3B -> unconnected-(U7-C1IN-/PSP1/RD1-Pad20)
- U7 pad 21: EN2/3 -> /S_PROG
- U7 pad 22: B_Up -> /S_INT
- U7 pad 24: /S_PROG -> B_Up
- U7 pad 34: /S_INT -> unconnected-(U7-RB1/INT1/AN8-Pad34)
- U7 pad 37: unconnected-(U7-RB4/KBI0/AN9-Pad37) -> Intermitente
- U7 pad 38: unconnected-(U7-RB5/KBI1/PGM-Pad38) -> Calentador
- U7 pad 5: Calentador -> IN1A
- U7 pad 6: unconnected-(U7-RA4/TOCKI-Pad6) -> EN1
- U7 pad 7: unconnected-(U7-RA5/ANA4/~{SS}/HLVDIN-Pad7) -> IN1B
- U7 pad 8: unconnected-(U7-AN5/~{RD}/RE0-Pad8) -> IN2/3A
- U7 pad 9: Intermitente -> EN2/3
Routing:
- net Vcc: track 64.4 -> 0.00 mm, vias 7 -> 0
- net GND: track 57.2 -> 1.44 mm, vias 77 -> 0
- net FiCa_A: track 11.1 -> 51.0 mm
- net /Motor23B: track 8.41 -> 45.9 mm
- net /S_INT: track 39.7 -> 4.48 mm, vias 2 -> 0
- net /Motor1A: track 24.6 -> 58.0 mm, vias 2 -> 0
- net Vdd: track 29.8 -> 0.00 mm
- net AngleMort: track 24.6 -> 0.00 mm
- net Net-(U6A--): track 30.9 -> 6.96 mm, vias 2 -> 0
- net Tx: track 23.5 -> 0.00 mm, vias 3 -> 0
- net Intermitente: track 23.0 -> 0.00 mm, vias 2 -> 0
- net /Motor1B: track 22.8 -> 45.7 mm, vias 2 -> 0
- net Net-(D5-A): track 21.1 -> 0.00 mm
- net FiCa_B: track 17.0 -> 37.2 mm, vias 2 -> 0
- net Calentador: track 20.0 -> 0.00 mm, vias 2 -> 0
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- added copper zone on F.Cu, net Vdd
- removed copper zone on F.Cu, net Vcc
Other:
- board size 96.5 x 85 mm -> 106.9 x 94.3 mm

Commit message: planos vcc
Parts:
- removed R6: 60, Resistor_SMD:R_0805_2012Metric_Pad1.20x1.40mm_HandSolder
- C11, C15, C16, C21, C22: moved to F.Cu
- moved REF** 266.0 mm to (189.3, 53.1)
- moved C15 223.7 mm to (138.7, 56.9), turned to 90 degrees
- moved C21 218.3 mm to (141.2, 56.9), turned to 90 degrees
- moved R23 216.8 mm to (135.6, 69.0), turned to 0 degrees
- moved Q2 216.1 mm to (134.9, 66.8)
- moved SW9 215.9 mm to (138.7, 61.0)
- moved D5 215.0 mm to (135.0, 53.9)
- moved C19 195.6 mm to (105.7, 64.6), turned to 90 degrees
- moved C20 193.3 mm to (108.4, 63.1)
- moved C3 192.5 mm to (98.7, 67.9)
- moved C14 191.1 mm to (117.1, 93.6)
- moved C9 190.8 mm to (127.9, 88.9)
- moved C17 187.7 mm to (156.4, 61.7), turned to 180 degrees
- moved C11 186.1 mm to (159.6, 116.5), turned to 180 degrees
- moved D4 178.9 mm to (90.1, 61.9)
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Connections:
- U7 pad 17: Act_Rele_M2/M3 -> unconnected-(U7-CCP1/RC2-Pad17)
- U7 pad 19: unconnected-(U7-C1IN+/PSP0/RD0-Pad19) -> Act_Rele_M2/M3
- U7 pad 20: unconnected-(U7-C1IN-/PSP1/RD1-Pad20) -> Intermitente
- U7 pad 37: Intermitente -> unconnected-(U7-RB4/KBI0/AN9-Pad37)
Routing:
- net AngleMort: track 0.00 -> 34.9 mm
- net /V_6: track 4.94 -> 25.8 mm
- net Tx: track 0.00 -> 20.8 mm, vias 0 -> 2
- net MAN_MCLR: track 0.00 -> 20.6 mm
- net Rx: track 0.00 -> 18.6 mm, vias 0 -> 2
- net /CAN+: track 0.00 -> 14.5 mm
- net /M_calen: track 0.00 -> 14.5 mm
- net /CAN-: track 0.00 -> 14.4 mm
- net PGC: track 0.00 -> 13.7 mm
- net Vcc: track 0.00 -> 13.5 mm, vias 0 -> 4
- net CANTX: track 0.00 -> 12.2 mm
- net Net-(U7-OSC1/CLKI/RA7): track 0.00 -> 11.7 mm
- net Net-(U7-OSC2/CLKO/RA6): track 0.00 -> 11.7 mm
- net PGD: track 0.00 -> 11.3 mm
- net Net-(D3-A): track 0.00 -> 11.0 mm
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- added copper zone on F.Cu, net Vcc
- removed copper zone on B.Cu, net GND
- removed copper zone on B.Cu, net GNDPWR
Other:
- board size 106.9 x 94.3 mm -> 106.6 x 91.3 mm

Commit message: Ns pero creo que asi se queda
Parts:
- moved R8 204.5 mm to (161.4, 134.3), turned to -90 degrees
- moved D2 1.65 mm to (147.1, 132.5)
- moved R20 1.65 mm to (142.9, 132.5)
- moved R18 0.90 mm to (161.0, 112.0)
- moved C11 0.85 mm to (158.8, 116.5)
- moved C15 0.53 mm to (138.2, 56.8)
- moved U3 0.07 mm to (177.9, 122.7)
Routing:
- net GND: track 0.00 -> 57.8 mm, vias 0 -> 81
- net GNDPWR: track 0.00 -> 15.6 mm, vias 0 -> 13
- net /M_Inter: track 7.91 -> 13.0 mm
- net Net-(U6B-+): track 7.36 -> 10.1 mm
- net Vcc: track 13.5 -> 15.7 mm, vias 4 -> 6
- net Net-(D2-A): track 0.00 -> 2.15 mm
- net IN1B: track 44.8 -> 46.2 mm
- net IN1A: track 47.8 -> 48.0 mm, vias 0 -> 1
- added copper zone on B.Cu, net GND
- added copper zone on B.Cu, net GNDPWR
Other:
- board size 106.6 x 91.3 mm -> 107.2 x 91.8 mm

Commit message: Asi se queda demomento
Parts:
- moved J2 0.76 mm to (98.5, 115.8)
- moved C22 0.68 mm to (104.3, 129.8)
- moved REF** 0.65 mm to (189.4, 52.5)
- moved REF** 0.44 mm to (90.0, 52.6)
- moved REF** 0.30 mm to (90.1, 137.3)
- moved U3 0.11 mm to (177.9, 122.8)
- moved C6 0.05 mm to (166.9, 82.8)
Routing:
- net GND: track 57.8 -> 60.4 mm, vias 81 -> 86
- net Vcc: track 15.7 -> 13.4 mm
- net /CAN+: track 14.5 -> 13.7 mm
- net /CAN-: track 14.4 -> 13.7 mm
Other:
- board size 107.2 x 91.8 mm -> 106.5 x 91.8 mm

Commit message: ghty
Parts:
- moved R24 0.30 mm to (154.2, 65.7)
- moved C17 0.23 mm to (156.4, 61.5)
Routing:
- net Vcc: track 13.4 -> 6.81 mm, vias 6 -> 15
- net Act_Rele_M2/M3: vias 2 -> 0
- net IN1A: vias 1 -> 0
- added copper zone on B.Cu, net Vcc
Changed lines of the file:
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@@
 	(footprint "Capacitor_SMD:C_1206_3216Metric_Pad1.33x1.80mm_HandSolder"
 		(layer "F.Cu")
-		(at 156.4375 61.725 180)
+		(at 156.4383 61.4914 180)
 		(descr "Capacitor SMD 1206 (3216 Metric), square (rectangular) end terminal, IPC_7351 nominal with elongated pad for handsoldering. (Body size source: IPC-SM-782 page 76, https://www.pcb-3d.com/wordpress/wp-content/uploads/ipc-sm-782a_amendment_1_and_2.pdf), generated with kicad-footprint-generator")
 		(tags "capacitor handsolder")
@@
 	(footprint "Resistor_SMD:R_0805_2012Metric_Pad1.20x1.40mm_HandSolder"
 		(layer "F.Cu")
-		(at 154.1584 65.379 180)
+		(at 154.1584 65.6762 180)
 		(descr "Resistor SMD 0805 (2012 Metric), square (rectangular) end terminal, IPC_7351 nominal with elongated pad for handsoldering. (Body size source: IPC-SM-782 page 72, https://www.pcb-3d.com/wordpress/wp-content/uploads/ipc-sm-782a_amendment_1_and_2.pdf), generated with kicad-footprint-generator")
 		(tags "resistor handsolder")
@@
 	)
 	(segment
-		(start 153.162 66.3956)
-		(end 153.162 64.3636)
+		(start 153.162 66.6928)
+		(end 153.162 64.6608)
 		(width 0.6)
 		(layer "F.Cu")
@@
 	)
 	(segment
-		(start 154.8892 62.9412)
-		(end 154.8892 60.5536)
+		(start 154.89 62.7076)
+		(end 154.89 60.32)
 		(width 0.6)
 		(layer "F.Cu")
@@
 	)
 	(via
-		(at 153.162 66.3956)
+		(at 153.162 66.6928)
 		(size 0.6)
 		(drill 0.2)
@@
 	)
 	(via
-		(at 153.2128 64.3128)
+		(at 153.2128 64.61)
 		(size 0.6)
 		(drill 0.2)
@@
 	)
 	(via
-		(at 154.8892 62.9412)
+		(at 154.89 62.7076)
 		(size 0.6)
 		(drill 0.2)
@@
 	)
 	(via
-		(at 154.94 60.5028)
+		(at 154.9408 60.2692)
 		(size 0.6)
 		(drill 0.2)
@@
 	)
 	(via
-		(at 162.2552 98.4504)
+		(at 154.55 100.62)
+		(size 0.6)
+		(drill 0.2)
+		(layers "F.Cu" "B.Cu")
+		(free yes)
+		(net 4)
+	)
+	(via
+		(at 162.16 97.5)
 		(size 0.6)
 		(drill 0.2)
@@
 	)
 	(via
-		(at 158.9024 99.0092)
+		(at 159.07 97.54)
+		(size 0.6)
+		(drill 0.2)
+		(layers "F.Cu" "B.Cu")
+		(free yes)
+		(net 4)
+	)
+	(via
+		(at 154.04 100.16)
+		(size 0.6)
+		(drill 0.2)
+		(layers "F.Cu" "B.Cu")
+		(free yes)
+		(net 4)
+	)
+	(via
+		(at 164.2 97.46)
+		(size 0.6)
+		(drill 0.2)
+		(layers "F.Cu" "B.Cu")
+		(free yes)
+		(net 4)
+	)
+	(via
+		(at 162.18 99.02)
+		(size 0.6)
+		(drill 0.2)
+		(layers "F.Cu" "B.Cu")
+		(free yes)
+		(net 4)
+	)
+	(via
+		(at 164.19 98.24)
+		(size 0.6)
+		(drill 0.2)
+		(layers "F.Cu" "B.Cu")
+		(free yes)
+		(net 4)
+	)
+	(via
+		(at 159.09 99.01)
 		(size 0.6)
 		(drill 0.2)
@@
 	)
 	(via
-		(at 154.686 100.4824)
+		(at 162.17 98.31)
 		(size 0.6)
 		(drill 0.2)
@@
 	)
 	(via
-		(at 163.9824 98.4504)
+		(at 164.17 99.01)
 		(size 0.6)
 		(drill 0.2)
@@
 		(net 4)
 	)
-	(segment
-		(start 156.1592 99.0092)
-		(end 158.9024 99.0092)
-		(width 0.2)
-		(layer "B.Cu")
+	(via
+		(at 159.07 98.25)
+		(size 0.6)
+		(drill 0.2)
+		(layers "F.Cu" "B.Cu")
+		(free yes)
 		(net 4)
 	)
-	(segment
-		(start 114.8488 95.1748)
-		(end 117.0748 95.1748)
-		(width 0.2)
-		(layer "B.Cu")
+	(via
+		(at 153.53 99.61)
+		(size 0.6)
+		(drill 0.2)
+		(layers "F.Cu" "B.Cu")
+		(free yes)
+		(net 4)
+	)
+	(via
+		(at 155.08 101.15)
+		(size 0.6)
+		(drill 0.2)
+		(layers "F.Cu" "B.Cu")
+		(free yes)
 		(net 4)
 	)
 	(segment
-		(start 162.2552 98.4504)
-		(end 163.9824 98.4504)
+		(start 114.8488 95.1748)
+		(end 117.0748 95.1748)
 		(width 0.2)
 		(layer "B.Cu")
@@
 	)
 	(segment
-		(start 154.686 100.4824)
-		(end 156.1592 99.0092)
-		(width 0.2)
-		(layer "B.Cu")
-		(net 4)
-	)
-	(segment
 		(start 117.0748 95.1748)
 		(end 117.075 95.175)
@@
 	)
 	(segment
-		(start 176.15 117.6)
-		(end 176.15 118.15)
-		(width 0.2)
-		(layer "F.Cu")
-		(net 8)
-	)
-	(segment
 		(start 165.8 123.2)
 		(end 165.8 123.9625)
@@
 	)
 	(segment
-		(start 175.701 118.599)
-		(end 171.351 118.599)
+		(start 168 122.95)
+		(end 166.05 122.95)
 		(width 0.2)
 		(layer "F.Cu")
@@
 	)
 	(segment
-		(start 168 122.95)
-		(end 166.05 122.95)
+		(start 171.351 118.599)
+		(end 168 121.95)
 		(width 0.2)
 		(layer "F.Cu")
@@
 	(segment
 		(start 176.15 115)
-		(end 176.15 117.6)
+		(end 176.15 118.15)
 		(width 0.2)
 		(layer "F.Cu")
@@
 	)
 	(segment
-		(start 171.351 118.599)
-		(end 168 121.95)
+		(start 175.701 118.599)
+		(end 171.351 118.599)
 		(width 0.2)
 		(layer "F.Cu")
@@
 	)
 	(segment
-		(start 176.15 117.6)
-		(end 176.15 117.775)
+		(start 168 121.95)
+		(end 168 122.95)
 		(width 0.2)
 		(layer "F.Cu")
@@
 	)
 	(segment
-		(start 168 121.95)
-		(end 168 122.95)
-		(width 0.2)
-		(layer "F.Cu")
-		(net 8)
-	)
-	(segment
 		(start 179.5698 118.4302)
 		(end 179.5698 115.0694)
@@
 	)
 	(segment
-		(start 151.2932 70.826)
-		(end 151.2824 70.8152)
+		(start 131.14 70.826)
+		(end 152.115036 70.826)
 		(width 0.2)
 		(layer "F.Cu")
@@
 	)
 	(segment
-		(start 153.29073 69.1388)
-		(end 156.63953 65.79)
+		(start 157.151036 65.79)
+		(end 157.3524 65.79)
 		(width 0.2)
 		(layer "F.Cu")
@@
 	)
 	(segment
-		(start 151.29756 70.826)
-		(end 151.2932 70.826)
+		(start 152.115036 70.826)
+		(end 157.151036 65.79)
 		(width 0.2)
 		(layer "F.Cu")
@@
 	)
 	(segment
-		(start 151.29756 70.826)
-		(end 131.14 70.826)
-		(width 0.2)
-		(layer "F.Cu")
-		(net 40)
-	)
-	(segment
 		(start 157.9084 65.234)
 		(end 157.3194 65.823)
@@
 	)
 	(segment
-		(start 156.63953 65.79)
-		(end 157.3524 65.79)
-		(width 0.2)
-		(layer "F.Cu")
-		(net 40)
-	)
-	(segment
-		(start 131.14 70.826)
-		(end 130.0888 69.7748)
+		(start 130.0888 69.7748)
+		(end 131.14 70.826)
 		(width 0.2)
 		(layer "F.Cu")
@@
 	)
 	(segment
-		(start 152.9588 69.1388)
-		(end 153.29073 69.1388)
-		(width 0.2)
-		(layer "F.Cu")
-		(net 40)
-	)
-	(via
-		(at 152.9588 69.1388)
-		(size 0.6)
-		(drill 0.2)
-		(layers "F.Cu" "B.Cu")
-		(net 40)
-	)
-	(via
-		(at 151.2824 70.8152)
-		(size 0.6)
-		(drill 0.2)
-		(layers "F.Cu" "B.Cu")
-		(net 40)
-	)
-	(segment
-		(start 151.2824 70.8152)
-		(end 152.9588 69.1388)
-		(width 0.2)
-		(layer "B.Cu")
-		(net 40)
-	)
-	(segment
 		(start 132.6152 67.2348)
 		(end 133.5 66.35)
@@
 	)
 	(segment
-		(start 169.7 102.75)
-		(end 167.1152 105.3348)
+		(start 170.73 101.72)
+		(end 170.73 95.82)
 		(width 0.2)
 		(layer "F.Cu")
@@
 	)
 	(segment
-		(start 167.1152 105.3348)
-		(end 130.0888 105.3348)
+		(start 130.0888 105.3348)
+		(end 167.1152 105.3348)
 		(width 0.2)
 		(layer "F.Cu")
 		(net 69)
 	)
-	(via
-		(at 169.7 102.75)
-		(size 0.6)
-		(drill 0.2)
-		(layers "F.Cu" "B.Cu")
-		(net 69)
-	)
 	(segment
-		(start 170.73 95.82)
+		(start 167.1152 105.3348)
 		(end 170.73 101.72)
 		(width 0.2)
-		(layer "B.Cu")
-		(net 69)
-	)
-	(segment
-		(start 170.73 101.72)
-		(end 169.7 102.75)
-		(width 0.2)
-		(layer "B.Cu")
+		(layer "F.Cu")
 		(net 69)
 	)
@@
 	)
 	(zone
+		(net 4)
+		(net_name "Vcc")
+		(layer "B.Cu")
+		(hatch edge 0.5)
+		(priority 6)
+		(connect_pads
+			(clearance 0.5)
+		)
+		(min_thickness 0.25)
+		(filled_areas_thickness no)
+		(fill yes
+			(thermal_gap 0.5)
+			(thermal_bridge_width 0.5)
+		)
+		(polygon
+			(pts
+				(xy 152.61 99.56) (xy 154.95 101.93) (xy 157.27 99.63) (xy 164.92681 99.593843) (xy 164.873701 96.991517)
+				(xy 155.56 97.06) (xy 152.59 99.56) (xy 152.65 99.55) (xy 152.61 99.54)
+			)
+		)
+	)
+	(zone
 		(net 1)
 		(net_name "GND")
@@
 				(xy 166.05564 112.966837) (xy 170.4 112.789077) (xy 170.4 111.41222) (xy 183.029509 111.362489)
 				(xy 183.012506 105.530339) (xy 157.996416 105.706922) (xy 158.089006 97.453343) (xy 141.353793 97.335488)
-				(xy 140.97 83.0072) (xy 156.5148 83.5152) (xy 156.967602 59.5884) (xy 150.8 59.85)
+				(xy 140.97 83.0072) (xy 156.5148 83.5152) (xy 156.97521 59.186379) (xy 150.801724 59.448229)
 			)
 		)
@@
 				(xy 143.429388 57.2516) (xy 140.060082 57.2516) (xy 140.002844 51.356321) (xy 134.006002 51.2572)
 				(xy 133.955202 63.3476) (xy 142.485525 63.285704) (xy 142.438802 71.0184) (xy 150.751722 71.101947)
-				(xy 150.608329 60.047317) (xy 156.967602 59.5884) (xy 156.214975 83.923325) (xy 140.97 83.0072)
+				(xy 150.601124 59.491857) (xy 156.984835 59.031176) (xy 156.214975 83.923325) (xy 140.97 83.0072)
 				(xy 141.345312 97.018838) (xy 158.482912 97.139525) (xy 158.387888 105.610145) (xy 183.012232 105.436325)
 				(xy 183.029509 111.362489) (xy 170.5 111.411826) (xy 170.5 112.784985) (xy 165.955821 112.970921)

Commit message: correccion errores
Parts:
- added R6: 60, Resistor_SMD:R_0805_2012Metric_Pad1.20x1.40mm_HandSolder, F.Cu at (107.0, 115.2)
- moved J7 91.6 mm to (190.3, 130.5), turned to 90 degrees
- moved C22 80.8 mm to (183.7, 114.8)
- moved C16 78.6 mm to (187.4, 121.4), turned to 0 degrees
- moved SW8 74.1 mm to (183.0, 122.1), turned to -90 degrees
- moved D3 73.2 mm to (185.2, 117.6), turned to 180 degrees
- moved R22 69.0 mm to (178.0, 114.0), turned to 0 degrees
- moved Q3 63.1 mm to (175.1, 114.7)
- moved D2 41.1 mm to (107.2, 122.7), turned to 0 degrees
- moved R8 33.1 mm to (182.9, 109.0), turned to 0 degrees
- moved R20 33.1 mm to (111.4, 122.7), turned to 180 degrees
- moved C1 27.1 mm to (170.9, 138.1), turned to 90 degrees
- moved U3 23.1 mm to (157.1, 133.0), turned to 180 degrees
- moved D1 21.3 mm to (171.1, 130.6), turned to 90 degrees
- moved C2 2.84 mm to (155.4, 121.8), turned to -90 degrees
- moved J10 1.96 mm to (189.9, 108.7)
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Connections:
- U7 pad 38: Calentador -> AngleMort
- U7 pad 4: AngleMort -> Calentador
Routing:
- net Calentador: track 8.86 -> 50.2 mm
- net AngleMort: track 34.7 -> 13.3 mm
- net /CAN-: track 13.7 -> 28.2 mm
- net /CAN+: track 13.7 -> 28.2 mm
- net GND: track 60.4 -> 64.5 mm, vias 86 -> 87
- net Net-(U3-FB): track 19.0 -> 15.0 mm
- net Net-(D1-K): track 19.4 -> 16.6 mm
- net /V_6: track 25.8 -> 27.4 mm
- net GNDPWR: track 15.6 -> 17.1 mm, vias 13 -> 14
- net /M_calen: track 14.5 -> 13.1 mm
- net Net-(Q3-E): track 1.55 -> 2.93 mm
- net IN1A: track 48.0 -> 48.3 mm, vias 0 -> 1
- net Vcc: track 6.81 -> 7.03 mm, vias 15 -> 11
Other:
- board size 106.5 x 91.8 mm -> 108.3 x 91.8 mm

Commit message: De to
Parts:
- added C23: 100n, Capacitor_SMD:C_0805_2012Metric_Pad1.18x1.45mm_HandSolder, F.Cu at (108.1, 72.1)
- added R25: 1K, Resistor_SMD:R_0805_2012Metric_Pad1.20x1.40mm_HandSolder, F.Cu at (111.0, 67.4)
- added R26: 1K, Resistor_SMD:R_0805_2012Metric_Pad1.20x1.40mm_HandSolder, F.Cu at (111.0, 71.2)
- added U8: LSF0002, PracticasKiCad:LSF0002, F.Cu at (108.3, 69.2)
- R10, R11: value 2k2 -> 1K; footprint Resistor_SMD:R_1206_3216Metric_Pad1.30x1.75mm_HandSolder -> Resistor_SMD:R_0805_2012Metric_Pad1.20x1.40mm_HandSolder
- SW2: value SW_Push -> UN/FOLD
- SW3: value SW_Push -> HEAT
- SW4: value SW_Push -> UP
- SW5: value SW_Push -> DOWN
- SW6: value SW_Push -> LEFT
- SW7: value SW_Push -> RIGHT
- U10: footprint Package_TO_SOT_SMD:TO-252-3_TabPin2 -> Package_TO_SOT_SMD:TO-263-3_TabPin2
- moved R10 24.5 mm to (105.2, 71.2), turned to 90 degrees
- moved R21 10.5 mm to (97.4, 56.5)
- moved D4 10.5 mm to (97.4, 54.3)
- moved R11 8.49 mm to (105.2, 67.4), turned to -90 degrees
- moved C19 8.01 mm to (97.9, 66.6)
- moved C20 8.01 mm to (100.6, 65.1)
- moved U1 8.01 mm to (101.6, 69.6)
- moved C3 8.01 mm to (91.0, 69.9)
- moved R3 8.01 mm to (98.5, 72.4)
- moved U2 8.01 mm to (94.3, 69.1)
- moved C5 5.68 mm to (142.2, 132.1)
- moved C4 5.07 mm to (146.3, 133.1)
- moved C6 3.35 mm to (167.7, 79.5)
- moved U10 2.17 mm to (143.5, 119.9)
- moved R9 1.89 mm to (134.2, 119.2)
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Connections:
- R10 pad 2: /S_SCL -> Net-(U1-SCL)
- R11 pad 2: /S_SDA -> Net-(U1-SDA)
- U1 pad 2: /S_SCL -> Net-(U1-SCL)
- U1 pad 4: /S_SDA -> Net-(U1-SDA)
Routing:
- net /S_PROG: track 4.09 -> 14.7 mm
- net /S_INT: track 4.48 -> 12.7 mm, vias 0 -> 1
- net Net-(U1-SCL): track 0.00 -> 5.44 mm
- net Vdd: track 0.00 -> 5.42 mm, vias 0 -> 2
- net /V_6: track 27.4 -> 32.3 mm
- net Net-(U1-SDA): track 0.00 -> 4.72 mm
- net /Motor1B: track 45.7 -> 50.4 mm
- net GND: track 64.5 -> 69.1 mm, vias 87 -> 90
- net /Motor1A: track 58.0 -> 61.3 mm
- net /S_SCL: track 27.5 -> 24.7 mm
- net /Motor23A: track 39.2 -> 41.6 mm
- net /Motor23B: track 45.9 -> 48.4 mm
- net /S_SDA: track 10.8 -> 8.77 mm
- net MAN_MCLR: track 20.6 -> 18.7 mm
- net Rx: track 18.6 -> 17.0 mm, vias 2 -> 0
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
Commit message: hgy
Other:
- board text added: "Projecte_Retrovisors_2025 Ines Fernandes Raul Robres Engenyeria Electrònica de Telecomunicació UB"
Changed lines of the file:
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@@
+	)
+	(gr_rect
+		(start 99.45 131.05)
+		(end 136 138.1)
+		(stroke
+			(width 0.1)
+			(type default)
+		)
+		(fill no)
+		(layer "F.SilkS")
 	)
 	(gr_rect
@@
 			)
 			(justify left bottom)
+		)
+	)
+	(gr_text "Projecte_Retrovisors_2025\nInes Fernandes\nRaul Robres\nEngenyeria Electrònica de Telecomunicació UB"
+		(at 100 137.75 0)
+		(layer "F.SilkS")
+		(effects
+			(font
+				(size 1 1)
+				(thickness 0.1)
+			)
+			(justify left bottom)
