File: DIMECRES_C_retrovisors.kicad_pcb (KiCad board)
At the start: 2 copper layers, 108.3 x 91.8 mm, 100 parts, among them J10 Vbat, J2 DE9_Pins, J3 Conn_01x05_Pin, J4 Motor3, J5 DE9_Pins, J6 Intermitente, J7 Calentador, J8 Motor2, J9 Motor1, Q1 DTC144E, Q2 DTC144E, Q3 DTC144E, SW1 SW_DPDT_G6S, SW10 SW_Push, SW2 UN/FOLD, SW3 HEAT, SW4 UP, SW5 DOWN, SW6 LEFT, SW7 RIGHT, SW8 FN01B, SW9 FN01B, U1 CH201, U10 LM1117DT-5.0, U2 ADM7160, U3 LM2596S-ADJ, U4 L298N, U5 MCP2551-I-SN, U6 ADA4511-2, U7 PIC18F4480-IP, U8 LSF0002, Y1 Crystal

Commit message: .,.
Parts:
- removed R8: 0, Resistor_SMD:R_0805_2012Metric_Pad1.20x1.40mm_HandSolder
- moved C20 0.42 mm to (100.8, 64.7)
Connections:
- net Net-(D1-K) renamed /OUT_BUCK
- net Net-(D3-A) renamed /Tran_Cal
- net Net-(D5-A) renamed /Tran_Int
- net Net-(U1-SCL) renamed /SCL1
- net Net-(U1-SDA) renamed /SDA1
- net Net-(U3-FB) renamed /FB
- net Net-(U6A-+) renamed /OPA_P
- net Net-(U6A--) renamed /OPA_N
- net Net-(U6B-+) renamed /OPB_P
- net Net-(U6B--) renamed /OPB_N
- net Net-(U7-OSC1/CLKI/RA7) renamed /OSC1
- net Net-(U7-OSC2/CLKO/RA6) renamed /OSC2
- C15 pad 2: GNDPWR -> GND
- C16 pad 2: GNDPWR -> GND
- C6 pad 2: GNDPWR -> GND
- C8 pad 2: GNDPWR -> GND
- D11 pad 2: GNDPWR -> GND
- D12 pad 2: GNDPWR -> GND
- D13 pad 2: GNDPWR -> GND
- D14 pad 2: GNDPWR -> GND
- J10 pad 2: GNDPWR -> GND
- J6 pad 2: GNDPWR -> GND
- J7 pad 2: GNDPWR -> GND
- R12 pad 1: GNDPWR -> GND
- R17 pad 1: GNDPWR -> GND
- R4 pad 2: GNDPWR -> GND
- R5 pad 2: GNDPWR -> GND
- U4 pad 8: GNDPWR -> GND
Routing:
- net GNDPWR: track 17.1 -> 0.00 mm, vias 14 -> 0
- net GND: track 69.1 -> 80.6 mm, vias 90 -> 104
- removed copper zone on B.Cu, net GNDPWR

Commit message: .
Parts:
- C21, C22: footprint Capacitor_SMD:C_1206_3216Metric_Pad1.33x1.80mm_HandSolder -> Capacitor_SMD:C_0805_2012Metric_Pad1.18x1.45mm_HandSolder
- C6: value 470U -> 470u
- J2, J5: footprint Connector_Dsub:DSUB-9_Socket_Horizontal_P2.77x2.54mm_EdgePinOffset9.40mm -> Connector_Dsub:DSUB-9_Socket_Vertical_P2.77x2.84mm_MountingHoles
- L1: footprint Inductor_SMD:L_1206_3216Metric_Pad1.22x1.90mm_HandSolder -> Inductor_SMD:L_0805_2012Metric_Pad1.05x1.20mm_HandSolder
- R9: footprint LED_SMD:LED_1206_3216Metric_Pad1.42x1.75mm_HandSolder -> Resistor_SMD:R_1206_3216Metric_Pad1.30x1.75mm_HandSolder
- moved J2 7.05 mm to (95.6, 122.2)
- moved J5 3.30 mm to (111.7, 58.2)
- moved C20 1.13 mm to (99.9, 65.4)
- moved C19 0.88 mm to (97.5, 67.4)
- moved C22 0.47 mm to (184.1, 114.9)
- moved L1 0.44 mm to (171.0, 124.9)
- moved C21 0.40 mm to (141.2, 57.3)
- moved U1 0.35 mm to (101.8, 69.9)
- moved R9 0.09 mm to (134.2, 119.1)
Routing:
- net /CAN+: track 28.2 -> 33.0 mm
- net /CAN-: track 28.2 -> 33.0 mm
- net Rx: track 17.0 -> 20.3 mm
- net Tx: track 20.7 -> 22.7 mm
- net /OUT_BUCK: track 16.6 -> 18.0 mm
- net GND: track 80.6 -> 80.9 mm, vias 104 -> 105

Commit message: muchas cosas a ya...
Changed lines of the file:
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@@
 			)
 		)
-		(property "LSCS" ""
+		(property "LSCS" " C107150"
 			(at 0 0 180)
 			(unlocked yes)
@@
 			)
 		)
-		(property "LSCS" ""
+		(property "LSCS" " C107150"
 			(at 0 0 90)
 			(unlocked yes)
@@
 	(footprint "Capacitor_SMD:C_1206_3216Metric_Pad1.33x1.80mm_HandSolder"
 		(layer "B.Cu")
-		(at 117.075 93.6125 90)
+		(at 107.9675 108.42)
 		(descr "Capacitor SMD 1206 (3216 Metric), square (rectangular) end terminal, IPC_7351 nominal with elongated pad for handsoldering. (Body size source: IPC-SM-782 page 76, https://www.pcb-3d.com/wordpress/wp-content/uploads/ipc-sm-782a_amendment_1_and_2.pdf), generated with kicad-footprint-generator")
 		(tags "capacitor handsolder")
-		(property "Reference" "C14"
-			(at 0 1.85 90)
+		(property "Reference" "C10"
+			(at 0 1.85 0)
 			(layer "B.SilkS")
 			(effects
@@
 		)
 		(property "Value" "100n"
-			(at 0 -1.85 90)
+			(at 0 -1.85 0)
 			(layer "B.Fab")
 			(effects
@@
 		)
 		(property "Datasheet" ""
-			(at 0 0 270)
+			(at 0 0 180)
 			(unlocked yes)
 			(layer "B.Fab")
@@
 		)
 		(property "Description" "Unpolarized capacitor"
-			(at 0 0 270)
+			(at 0 0 180)
 			(unlocked yes)
 			(layer "B.Fab")
@@
 		)
 		(property "LSCS" "C1945"
-			(at 0 0 90)
+			(at 0 0 180)
 			(unlocked yes)
 			(layer "B.Fab")
@@
 		)
 		(fp_line
-			(start 2.48 -1.15)
-			(end -2.48 -1.15)
+			(start -2.48 -1.15)
+			(end -2.48 1.15)
 			(stroke
 				(width 0.05)
@@
 		)
 		(fp_line
-			(start -2.48 -1.15)
-			(end -2.48 1.15)
+			(start -2.48 1.15)
+			(end 2.48 1.15)
 			(stroke
 				(width 0.05)
@@
 		)
 		(fp_line
-			(start 2.48 1.15)
-			(end 2.48 -1.15)
+			(start 2.48 -1.15)
+			(end -2.48 -1.15)
 			(stroke
 				(width 0.05)
@@
 		)
 		(fp_line
-			(start -2.48 1.15)
-			(end 2.48 1.15)
+			(start 2.48 1.15)
+			(end 2.48 -1.15)
 			(stroke
 				(width 0.05)
@@
 		)
 		(fp_line
-			(start 1.6 -0.8)
-			(end -1.6 -0.8)
+			(start -1.6 -0.8)
+			(end -1.6 0.8)
 			(stroke
 				(width 0.1)
@@
 		)
 		(fp_line
-			(start -1.6 -0.8)
-			(end -1.6 0.8)
+			(start -1.6 0.8)
+			(end 1.6 0.8)
 			(stroke
 				(width 0.1)
@@
 		)
 		(fp_line
-			(start 1.6 0.8)
-			(end 1.6 -0.8)
+			(start 1.6 -0.8)
+			(end -1.6 -0.8)
 			(stroke
 				(width 0.1)
@@
 		)
 		(fp_line
-			(start -1.6 0.8)
-			(end 1.6 0.8)
+			(start 1.6 0.8)
+			(end 1.6 -0.8)
 			(stroke
 				(width 0.1)
@@
 		)
 		(fp_text user "${REFERENCE}"
-			(at 0 0 90)
+			(at 0 0 0)
 			(layer "B.Fab")
 			(effects
@@
 		)
 		(pad "1" smd roundrect
-			(at -1.5625 0 90)
+			(at -1.5625 0)
 			(size 1.325 1.8)
 			(layers "B.Cu" "B.Mask" "B.Paste")
@@
 		)
 		(pad "2" smd roundrect
-			(at 1.5625 0 90)
+			(at 1.5625 0)
 			(size 1.325 1.8)
 			(layers "B.Cu" "B.Mask" "B.Paste")
@@
 	(footprint "Capacitor_SMD:C_1206_3216Metric_Pad1.33x1.80mm_HandSolder"
 		(layer "B.Cu")
-		(at 107.9975 108.425)
+		(at 117.075 93.6125 90)
 		(descr "Capacitor SMD 1206 (3216 Metric), square (rectangular) end terminal, IPC_7351 nominal with elongated pad for handsoldering. (Body size source: IPC-SM-782 page 76, https://www.pcb-3d.com/wordpress/wp-content/uploads/ipc-sm-782a_amendment_1_and_2.pdf), generated with kicad-footprint-generator")
 		(tags "capacitor handsolder")
-		(property "Reference" "C10"
-			(at 0 1.85 0)
+		(property "Reference" "C14"
+			(at 0 1.85 90)
 			(layer "B.SilkS")
-			(hide yes)
 			(effects
 				(font
@@
 		)
 		(property "Value" "100n"
-			(at 0 -1.85 0)
+			(at 0 -1.85 90)
 			(layer "B.Fab")
 			(effects
@@
 		)
 		(property "Datasheet" ""
-			(at 0 0 180)
+			(at 0 0 270)
 			(unlocked yes)
 			(layer "B.Fab")
@@
 		)
 		(property "Description" "Unpolarized capacitor"
-			(at 0 0 180)
+			(at 0 0 270)
 			(unlocked yes)
 			(layer "B.Fab")
@@
 		)
 		(property "LSCS" "C1945"
-			(at 0 0 0)
+			(at 0 0 90)
 			(unlocked yes)
 			(layer "B.Fab")
@@
 		)
 		(fp_line
-			(start -2.48 -1.15)
-			(end -2.48 1.15)
+			(start 2.48 -1.15)
+			(end -2.48 -1.15)
 			(stroke
 				(width 0.05)
@@
 		)
 		(fp_line
-			(start -2.48 1.15)
-			(end 2.48 1.15)
+			(start -2.48 -1.15)
+			(end -2.48 1.15)
 			(stroke
 				(width 0.05)
@@
 		)
 		(fp_line
-			(start 2.48 -1.15)
-			(end -2.48 -1.15)
+			(start 2.48 1.15)
+			(end 2.48 -1.15)
 			(stroke
 				(width 0.05)
@@
 		)
 		(fp_line
-			(start 2.48 1.15)
-			(end 2.48 -1.15)
+			(start -2.48 1.15)
+			(end 2.48 1.15)
 			(stroke
 				(width 0.05)
@@
 		)
 		(fp_line
-			(start -1.6 -0.8)
-			(end -1.6 0.8)
+			(start 1.6 -0.8)
+			(end -1.6 -0.8)
 			(stroke
 				(width 0.1)
@@
 		)
 		(fp_line
-			(start -1.6 0.8)
-			(end 1.6 0.8)
+			(start -1.6 -0.8)
+			(end -1.6 0.8)
 			(stroke
 				(width 0.1)
@@
 		)
 		(fp_line
-			(start 1.6 -0.8)
-			(end -1.6 -0.8)
+			(start 1.6 0.8)
+			(end 1.6 -0.8)
 			(stroke
 				(width 0.1)
@@
 		)
 		(fp_line
-			(start 1.6 0.8)
-			(end 1.6 -0.8)
+			(start -1.6 0.8)
+			(end 1.6 0.8)
 			(stroke
 				(width 0.1)
@@
 		)
 		(fp_text user "${REFERENCE}"
-			(at 0 0 0)
+			(at 0 0 90)
 			(layer "B.Fab")
 			(effects
@@
 		)
 		(pad "1" smd roundrect
-			(at -1.5625 0)
+			(at -1.5625 0 90)
 			(size 1.325 1.8)
 			(layers "B.Cu" "B.Mask" "B.Paste")
@@
 		)
 		(pad "2" smd roundrect
-			(at 1.5625 0)
+			(at 1.5625 0 90)
 			(size 1.325 1.8)
 			(layers "B.Cu" "B.Mask" "B.Paste")
